Commit message: renaming macro "variables" for more clear assosiation

File: ros2_ws/src/libra/models/2dof_and_arm.urdf.xacro (robot description, xacro)
@@ -2,15 +2,20 @@
 <robot name="robot_arm" xmlns:xacro="http://www.ros.org/wiki/xacro">
     <xacro:property name="PI" value="3.14159265359"/>
-    <xacro:property name="d_2djnt_h_L" value="0.143"/>
-    <xacro:property name="d_2djnt_h_W" value="0.165"/>
-    <xacro:property name="d_2djnt_h_H" value="0.158"/>
-    <xacro:property name="d_2djnt_L" value="0.204"/>
-    <xacro:property name="d_2djnt_W" value="0.145"/>
-    <xacro:property name="d_2djnt_H" value="0.090"/>
+    <!-- 2-DoF Joint (active part) -->
+    <xacro:property name="d_2djnt_a_L" value="0.143"/>
+    <xacro:property name="d_2djnt_a_W" value="0.165"/>
+    <xacro:property name="d_2djnt_a_H" value="0.1565"/>
+    <!-- 2-DoF Joint (passive part) -->
+    <xacro:property name="d_2djnt_p_L" value="0.204"/>
+    <xacro:property name="d_2djnt_p_W" value="0.145"/>
+    <xacro:property name="d_2djnt_p_H" value="0.090"/>
+    <!-- 2-DoF-to-Arm Connector -->
     <xacro:property name="d_conn_L" value="0.076"/>
     <xacro:property name="d_conn_W" value="0.076"/>
     <xacro:property name="d_conn_H" value="0.076"/>
+    <!-- Arm Links -->
     <xacro:property name="d_L_len" value="0.900"/>
     <xacro:property name="d_L_rad" value="0.030"/>
+    <!-- Arm Joints -->
     <xacro:property name="d_J12_L" value="0.12914"/>
     <xacro:property name="d_J12_W" value="0.076"/>
@@ -19,20 +24,19 @@
     <xacro:property name="d_J3_W" value="0.15705"/>
     <xacro:property name="d_J3_H" value="0.076"/>
-    <xacro:property name="d_manip_mount_L" value="0.100"/>
-    <xacro:property name="d_manip_mount_W" value="0.070"/>
-    <xacro:property name="d_manip_mount_H" value="0.0935"/>
+    <!-- Arm Tip / Manipulator Mount -->
+    <xacro:property name="d_arm_tip_L" value="0.100"/>
+    <xacro:property name="d_arm_tip_W" value="0.070"/>
+    <xacro:property name="d_arm_tip_H" value="0.0935"/>
+    <!-- Manipulator Joints -->
     <xacro:property name="d_mj1_L" value="0.0405"/>
     <xacro:property name="d_mj1_W" value="0.0405"/>
     <xacro:property name="d_mj1_H" value="0.020"/>
-    <xacro:property name="d_mj2_L" value="0.058"/>
-    <xacro:property name="d_mj2_W" value="0.0307"/>
-    <xacro:property name="d_mj2_H" value="0.0436"/>
-    <xacro:property name="d_mj3_L" value="0.058"/>
-    <xacro:property name="d_mj3_W" value="0.0436"/>
-    <xacro:property name="d_mj3_H" value="0.0307"/>
+    <xacro:property name="d_mj23_L" value="0.058"/>
+    <xacro:property name="d_mj23_W" value="0.0307"/>
+    <xacro:property name="d_mj23_H" value="0.0436"/>
     <xacro:property name="m_L" value="0.395"/>
     <xacro:property name="m_J12" value="0.851"/>
     <xacro:property name="m_J3" value="0.982"/> <xacro:property name="m_conn" value="0.155"/>
-    <xacro:property name="m_2djnt_h" value="1.780"/> <xacro:property name="m_2djnt" value="1.780"/> <xacro:property name="m_mj" value="0.039"/> <xacro:property name="m_manip_mount" value="0.170"/>
+    <xacro:property name="m_2djnt_a" value="1.780"/> <xacro:property name="m_2djnt" value="1.780"/> <xacro:property name="m_mj" value="0.039"/> <xacro:property name="m_manip_mount" value="0.170"/>
     <material name="red">
         <color rgba="${200/255} ${30/255} ${30/255} 1"/>
@@ -101,9 +105,9 @@
     <link name="base_link"/>
     ---
-    <link name="2djnt_housing_link">
-        <visual>
-            <origin xyz="0 0 0" rpy="0 0 0"/>
-            <geometry>
-                <box size="${d_2djnt_h_L} ${d_2djnt_h_W} ${d_2djnt_h_H}"/>
+    <link name="2d_active_link">
+        <visual>
+            <origin xyz="0 0 0" rpy="0 0 0"/>
+            <geometry>
+                <box size="${d_2djnt_a_L} ${d_2djnt_a_W} ${d_2djnt_a_H}"/>
             </geometry>
             <material name="black"/>
@@ -112,28 +116,28 @@
             <origin xyz="0 0 0" rpy="0 0 0"/>
             <geometry>
-                <box size="${d_2djnt_h_L} ${d_2djnt_h_W} ${d_2djnt_h_H}"/>
+                <box size="${d_2djnt_a_L} ${d_2djnt_a_W} ${d_2djnt_a_H}"/>
             </geometry>
         </collision>
-        <xacro:box_inertia m="${m_2djnt_h}" x="${d_2djnt_h_L}" y="${d_2djnt_h_W}" z="${d_2djnt_h_H}"/>
-    </link>
-    <joint name="base_to_2djnt_housing" type="fixed">
+        <xacro:box_inertia m="${m_2djnt_a}" x="${d_2djnt_a_L}" y="${d_2djnt_a_W}" z="${d_2djnt_a_H}"/>
+    </link>
+    <joint name="base_to_2d_active" type="fixed">
         <parent link="base_link"/>
-        <child link="2djnt_housing_link"/>
-        <origin xyz="0 0 -${d_2djnt_h_H/2}" rpy="0 0 0"/>
-    </joint>
-    ---
-    <link name="2djnt_pitch_link"/>
-    <joint name="2djnt_pitch_joint" type="revolute">
-        <parent link="2djnt_housing_link"/>
-        <child link="2djnt_pitch_link"/>
-        <origin xyz="${-d_2djnt_h_L/2 - 0.059 + d_2djnt_L/2} 0 ${d_2djnt_h_H/2 - 0.080 - d_2djnt_H/2}" rpy="0 0 0"/>
+        <child link="2d_active_link"/>
+        <origin xyz="0 0 -${d_2djnt_a_H/2}" rpy="0 0 0"/>
+    </joint>
+    ---
+    <link name="2d_passive_pitch_link"/>
+    <joint name="2d_pitch_joint" type="revolute">
+        <parent link="2d_active_link"/>
+        <child link="2d_passive_pitch_link"/>
+        <origin xyz="${-d_2djnt_a_L/2 - 0.059 + d_2djnt_p_L/2} 0 ${d_2djnt_a_H/2 - 0.080 - d_2djnt_p_H/2}" rpy="0 0 0"/>
         <axis xyz="0 1 0"/>
         <limit lower="-${PI/2}" upper="${PI/2}" effort="100" velocity="1.0"/>
     </joint>
-    <link name="2djnt_link">
-        <visual>
-            <origin xyz="0 0 0" rpy="0 0 0"/>
-            <geometry>
-                <box size="${d_2djnt_L} ${d_2djnt_W} ${d_2djnt_H}"/>
+    <link name="2d_passive_link">
+        <visual>
+            <origin xyz="0 0 0" rpy="0 0 0"/>
+            <geometry>
+                <box size="${d_2djnt_p_L} ${d_2djnt_p_W} ${d_2djnt_p_H}"/>
             </geometry>
             <material name="red"/>
@@ -142,12 +146,12 @@
             <origin xyz="0 0 0" rpy="0 0 0"/>
             <geometry>
-                <box size="${d_2djnt_L} ${d_2djnt_W} ${d_2djnt_H}"/>
+                <box size="${d_2djnt_p_L} ${d_2djnt_p_W} ${d_2djnt_p_H}"/>
             </geometry>
         </collision>
-        <xacro:box_inertia m="${m_2djnt}" x="${d_2djnt_L}" y="${d_2djnt_W}" z="${d_2djnt_H}"/>
-    </link>
-    <joint name="2djnt_roll_joint" type="revolute">
-        <parent link="2djnt_pitch_link"/>
-        <child link="2djnt_link"/>
+        <xacro:box_inertia m="${m_2djnt}" x="${d_2djnt_p_L}" y="${d_2djnt_p_W}" z="${d_2djnt_p_H}"/>
+    </link>
+    <joint name="2d_roll_joint" type="revolute">
+        <parent link="2d_passive_pitch_link"/>
+        <child link="2d_passive_link"/>
         <origin xyz="0 0 0" rpy="0 0 0"/>
         <axis xyz="1 0 0"/>
@@ -155,5 +159,5 @@
     </joint>
     ---
-    <link name="connector_link">
+    <link name="2d_arm_connector_link">
         <visual>
             <origin xyz="0 0 0" rpy="0 0 0"/>
@@ -171,13 +175,13 @@
         <xacro:box_inertia m="${m_conn}" x="${d_conn_L}" y="${d_conn_W}" z="${d_conn_H}"/>
     </link>
-    <joint name="2djnt_to_connector" type="fixed">
-        <parent link="2djnt_link"/>
-        <child link="connector_link"/>
-        <origin xyz="${(d_2djnt_L/2 - 0.022) + d_conn_L/2} 0 ${d_2djnt_H/2 - 0.0225 - d_conn_H/2}" rpy="0 0 0"/>
+    <joint name="2d_passive_to_2d_arm_connector" type="fixed">
+        <parent link="2d_passive_link"/>
+        <child link="2d_arm_connector_link"/>
+        <origin xyz="${(d_2djnt_p_L/2 - 0.022) + d_conn_L/2} 0 ${d_2djnt_p_H/2 - 0.0225 - d_conn_H/2}" rpy="0 0 0"/>
     </joint>
     ---
     <xacro:arm_link_macro name="L1_link"/>
-    <joint name="connector_to_L1" type="fixed">
-        <parent link="connector_link"/>
+    <joint name="2d_arm_connector_to_L1" type="fixed">
+        <parent link="2d_arm_connector_link"/>
         <child link="L1_link"/>
         <origin xyz="${d_conn_L/2 + d_L_len/2} 0 0" rpy="0 0 0"/>
@@ -228,9 +232,9 @@
         <origin xyz="${(d_J3_L/2 - 0.04014) + d_L_len/2} ${d_J3_W/2 - 0.038} 0" rpy="0 0 0"/>
     </joint>
-    <link name="manip_mount_link">
-        <visual>
-            <origin xyz="0 0 0" rpy="0 0 0"/>
-            <geometry>
-                <box size="${d_manip_mount_L} ${d_manip_mount_W} ${d_manip_mount_H}"/>
+    <link name="arm_tip_link">
+        <visual>
+            <origin xyz="0 0 0" rpy="0 0 0"/>
+            <geometry>
+                <box size="${d_arm_tip_L} ${d_arm_tip_W} ${d_arm_tip_H}"/>
             </geometry>
             <material name="black"/>
@@ -239,13 +243,13 @@
             <origin xyz="0 0 0" rpy="0 0 0"/>
             <geometry>
-                <box size="${d_manip_mount_L} ${d_manip_mount_W} ${d_manip_mount_H}"/>
+                <box size="${d_arm_tip_L} ${d_arm_tip_W} ${d_arm_tip_H}"/>
             </geometry>
         </collision>
-        <xacro:box_inertia m="${m_manip_mount}" x="${d_manip_mount_L}" y="${d_manip_mount_W}" z="${d_manip_mount_H}"/>
-    </link>
-    <joint name="L4_to_manip_mount" type="fixed">
+        <xacro:box_inertia m="${m_manip_mount}" x="${d_arm_tip_L}" y="${d_arm_tip_W}" z="${d_arm_tip_H}"/>
+    </link>
+    <joint name="L4_to_arm_tip" type="fixed">
         <parent link="L4_link"/>
-        <child link="manip_mount_link"/>
-        <origin xyz="${d_L_len/2 + d_manip_mount_L/2} 0 ${0.042 - d_manip_mount_H/2}" rpy="0 0 0"/>
+        <child link="arm_tip_link"/>
+        <origin xyz="${d_L_len/2 + d_arm_tip_L/2} 0 ${0.042 - d_arm_tip_H/2}" rpy="0 0 0"/>
     </joint>
     ---
@@ -260,8 +264,8 @@
         <xacro:box_inertia m="${m_mj}" x="${d_mj1_L}" y="${d_mj1_W}" z="${d_mj1_H}"/>
     </link>
-    <joint name="mount_to_mj1" type="revolute">
-        <parent link="manip_mount_link"/>
+    <joint name="arm_tip_to_mj1" type="revolute">
+        <parent link="arm_tip_link"/>
         <child link="mj1_link"/>
-        <origin xyz="${(d_manip_mount_L/2 - 0.00875) - d_mj1_L/2} ${-d_manip_mount_W/2 - 0.0121 + d_mj1_W/2} ${(d_manip_mount_H/2 - 0.006) - d_mj1_H/2}" rpy="0 0 0"/>
+        <origin xyz="${(d_arm_tip_L/2 - 0.00875) - d_mj1_L/2} ${-d_arm_tip_W/2 - 0.0121 + d_mj1_W/2} ${(d_arm_tip_H/2 - 0.006) - d_mj1_H/2}" rpy="0 0 0"/>
         <axis xyz="0 1 0"/>
         <limit lower="-${PI/2}" upper="${PI/2}" effort="50" velocity="1.5"/>
@@ -270,15 +274,15 @@
         <visual>
             <geometry>
-                <box size="${d_mj2_L} ${d_mj2_W} ${d_mj2_H}"/>
+                <box size="${d_mj23_L} ${d_mj23_W} ${d_mj23_H}"/>
             </geometry>
             <material name="purple"/>
         </visual>
-        <collision><geometry><box size="${d_mj2_L} ${d_mj2_W} ${d_mj2_H}"/></geometry></collision>
-        <xacro:box_inertia m="${m_mj}" x="${d_mj2_L}" y="${d_mj2_W}" z="${d_mj2_H}"/>
+        <collision><geometry><box size="${d_mj23_L} ${d_mj23_W} ${d_mj23_H}"/></geometry></collision>
+        <xacro:box_inertia m="${m_mj}" x="${d_mj23_L}" y="${d_mj23_W}" z="${d_mj23_H}"/>
     </link>
     <joint name="mj1_to_mj2" type="revolute">
         <parent link="mj1_link"/>
         <child link="mj2_link"/>
-        <origin xyz="${(d_mj1_L/2 + 0.0295) - d_mj2_L/2} ${-d_mj1_W/2 - d_mj2_W/2} ${(d_mj1_H/2 + 0.0091) - d_mj2_H/2}" rpy="0 0 0"/>
+        <origin xyz="${(d_mj1_L/2 + 0.0295) - d_mj23_L/2} ${-d_mj1_W/2 - d_mj23_W/2} ${(d_mj1_H/2 + 0.0091) - d_mj23_H/2}" rpy="0 0 0"/>
         <axis xyz="0 0 1"/>
         <limit lower="-${PI/2}" upper="${PI/2}" effort="50" velocity="1.5"/>
@@ -287,21 +291,21 @@
         <visual>
             <geometry>
-                <box size="${d_mj3_L} ${d_mj3_W} ${d_mj3_H}"/>
+                <box size="${d_mj23_L} ${d_mj23_H} ${d_mj23_W}"/>
             </geometry>
             <material name="purple"/>
         </visual>
-        <collision><geometry><box size="${d_mj3_L} ${d_mj3_W} ${d_mj3_H}"/></geometry></collision>
-        <xacro:box_inertia m="${m_mj}" x="${d_mj3_L}" y="${d_mj3_W}" z="${d_mj3_H}"/>
+        <collision><geometry><box size="${d_mj23_L} ${d_mj23_H} ${d_mj23_W}"/></geometry></collision>
+        <xacro:box_inertia m="${m_mj}" x="${d_mj23_L}" y="${d_mj23_H}" z="${d_mj23_W}"/>
     </link>
     <joint name="mj2_to_mj3" type="revolute">
         <parent link="mj2_link"/>
         <child link="mj3_link"/>
-        <origin xyz="${(-d_mj2_L/2 + 0.00025) + d_mj3_L/2} ${d_mj2_W/2 + 0.0053 - d_mj3_W/2} ${d_mj2_H/2 + d_mj3_H/2}" rpy="0 0 0"/>
+        <origin xyz="${(-d_mj23_L/2 + 0.00025) + d_mj23_L/2} ${d_mj23_W/2 + 0.0053 - d_mj23_H/2} ${d_mj23_H/2 + d_mj23_W/2}" rpy="0 0 0"/>
         <axis xyz="0 1 0"/>
         <limit lower="-${PI/2}" upper="${PI/2}" effort="50" velocity="1.5"/>
     </joint>
-    <gazebo reference="2djnt_housing_link"><material>Gazebo/Black</material></gazebo>
-    <gazebo reference="2djnt_link"><material>Gazebo/Red</material></gazebo>
-    <gazebo reference="connector_link"><material>Gazebo/Black</material></gazebo>
+    <gazebo reference="2d_active_link"><material>Gazebo/Black</material></gazebo>
+    <gazebo reference="2d_passive_link"><material>Gazebo/Red</material></gazebo>
+    <gazebo reference="2d_arm_connector_link"><material>Gazebo/Black</material></gazebo>
     <gazebo reference="L1_link"><material>Gazebo/Gray</material></gazebo>
     <gazebo reference="J1_link"><material>Gazebo/Red</material></gazebo>
@@ -311,5 +315,5 @@
     <gazebo reference="J3_link"><material>Gazebo/Red</material></gazebo>
     <gazebo reference="L4_link"><material>Gazebo/Gray</material></gazebo>
-    <gazebo reference="manip_mount_link"><material>Gazebo/Black</material></gazebo>
+    <gazebo reference="arm_tip_link"><material>Gazebo/Black</material></gazebo>
     <gazebo reference="mj1_link"><material>Gazebo/Purple</material></gazebo>
     <gazebo reference="mj2_link"><material>Gazebo/Purple</material></gazebo>
