Commit message: added comments and renaming again for clarity - got some stuff mixed up

File: ros2_ws/src/libra/models/2dof_and_arm.urdf.xacro (robot description, xacro)
@@ -1,42 +1,49 @@
 <?xml version="1.0"?>
 <robot name="robot_arm" xmlns:xacro="http://www.ros.org/wiki/xacro">
+    <!-- ********************[ PROPERTIES ]******************** -->
+    <!-- Common -->
     <xacro:property name="PI" value="3.14159265359"/>
-    <!-- 2-DoF Joint (active part) -->
-    <xacro:property name="d_2djnt_a_L" value="0.143"/>
-    <xacro:property name="d_2djnt_a_W" value="0.165"/>
-    <xacro:property name="d_2djnt_a_H" value="0.1565"/>
-    <!-- 2-DoF Joint (passive part) -->
-    <xacro:property name="d_2djnt_p_L" value="0.204"/>
-    <xacro:property name="d_2djnt_p_W" value="0.145"/>
-    <xacro:property name="d_2djnt_p_H" value="0.090"/>
+    <!-- 2-DoF Joint (static part - "passive") -->
+    <xacro:property name="d_2djnt_p_L" value="0.143"/>
+    <xacro:property name="d_2djnt_p_W" value="0.165"/>
+    <xacro:property name="d_2djnt_p_H" value="0.1565"/>
+    <xacro:property name="m_2djnt_p" value="2.056"/>
+    <!-- 2-DoF Joint (moved part - "active") -->
+    <xacro:property name="d_2djnt_a_L" value="0.204"/>
+    <xacro:property name="d_2djnt_a_W" value="0.145"/>
+    <xacro:property name="d_2djnt_a_H" value="0.090"/>
+    <xacro:property name="m_2djnt_a" value="1.317"/>
     <!-- 2-DoF-to-Arm Connector -->
     <xacro:property name="d_conn_L" value="0.076"/>
     <xacro:property name="d_conn_W" value="0.076"/>
     <xacro:property name="d_conn_H" value="0.076"/>
+    <xacro:property name="m_conn" value="0.187"/>
     <!-- Arm Links -->
     <xacro:property name="d_L_len" value="0.900"/>
     <xacro:property name="d_L_rad" value="0.030"/>
+    <xacro:property name="m_L" value="0.395"/>
     <!-- Arm Joints -->
     <xacro:property name="d_J12_L" value="0.12914"/>
     <xacro:property name="d_J12_W" value="0.076"/>
     <xacro:property name="d_J12_H" value="0.15705"/>
+    <xacro:property name="m_J12" value="0.851"/>
     <xacro:property name="d_J3_L" value="0.14614"/>
     <xacro:property name="d_J3_W" value="0.15705"/>
     <xacro:property name="d_J3_H" value="0.076"/>
+    <xacro:property name="m_J3" value="0.982"/>
     <!-- Arm Tip / Manipulator Mount -->
     <xacro:property name="d_arm_tip_L" value="0.100"/>
     <xacro:property name="d_arm_tip_W" value="0.070"/>
     <xacro:property name="d_arm_tip_H" value="0.0935"/>
+    <xacro:property name="m_arm_tip" value="0.170"/>
     <!-- Manipulator Joints -->
-    <xacro:property name="d_mj1_L" value="0.0405"/>
-    <xacro:property name="d_mj1_W" value="0.0405"/>
-    <xacro:property name="d_mj1_H" value="0.020"/>
-    <xacro:property name="d_mj23_L" value="0.058"/>
-    <xacro:property name="d_mj23_W" value="0.0307"/>
-    <xacro:property name="d_mj23_H" value="0.0436"/>
-    <xacro:property name="m_L" value="0.395"/>
-    <xacro:property name="m_J12" value="0.851"/>
-    <xacro:property name="m_J3" value="0.982"/> <xacro:property name="m_conn" value="0.155"/>
-    <xacro:property name="m_2djnt_a" value="1.780"/> <xacro:property name="m_2djnt" value="1.780"/> <xacro:property name="m_mj" value="0.039"/> <xacro:property name="m_manip_mount" value="0.170"/>
+    <xacro:property name="d_MJ1_L" value="0.0405"/>
+    <xacro:property name="d_MJ1_W" value="0.0405"/>
+    <xacro:property name="d_MJ1_H" value="0.020"/>
+    <xacro:property name="d_MJ23_L" value="0.058"/>
+    <xacro:property name="d_MJ23_W" value="0.0307"/>
+    <xacro:property name="d_MJ23_H" value="0.0436"/>
+    <xacro:property name="m_MJ" value="0.039"/>
+    <!-- ********************[ MATERIALS ]******************** -->
     <material name="red">
         <color rgba="${200/255} ${30/255} ${30/255} 1"/>
@@ -51,4 +58,5 @@
         <color rgba="${150/255} ${50/255} ${200/255} 1"/>
     </material>
+    <!-- ********************[ MACROS ]******************** -->
     <xacro:macro name="box_inertia" params="m x y z">
         <inertial>
@@ -103,7 +111,41 @@
         </link>
     </xacro:macro>
+    <!-- ********************[ LINKS ]******************** -->
+    <!-- Base Link -->
     <link name="base_link"/>
     ---
-    <link name="2d_active_link">
+    <!-- 2-DoF Joint (passive part) -->
+    <link name="2d_passive_link">
+        <visual>
+            <origin xyz="0 0 0" rpy="0 0 0"/>
+            <geometry>
+                <box size="${d_2djnt_p_L} ${d_2djnt_p_W} ${d_2djnt_p_H}"/>
+            </geometry>
+            <material name="black"/>
+        </visual>
+        <collision>
+            <origin xyz="0 0 0" rpy="0 0 0"/>
+            <geometry>
+                <box size="${d_2djnt_p_L} ${d_2djnt_p_W} ${d_2djnt_p_H}"/>
+            </geometry>
+        </collision>
+        <xacro:box_inertia m="${m_2djnt_p}" x="${d_2djnt_p_L}" y="${d_2djnt_p_W}" z="${d_2djnt_p_H}"/>
+    </link>
+    <joint name="base_to_2d" type="fixed">
+        <parent link="base_link"/>
+        <child link="2d_passive_link"/>
+        <origin xyz="0 0 -${d_2djnt_p_H/2}" rpy="0 0 0"/>
+    </joint>
+    ---
+    <!-- 2-DoF Joint (active part) -->
+    <link name="2d_active_pitch_link"/>
+    <joint name="2d_pitch_joint" type="revolute">
+        <parent link="2d_passive_link"/>
+        <child link="2d_active_pitch_link"/>
+        <origin xyz="${-d_2djnt_p_L/2 - 0.059 + d_2djnt_a_L/2} 0 ${d_2djnt_p_H/2 - 0.080 - d_2djnt_a_H/2}" rpy="0 0 0"/>
+        <axis xyz="0 1 0"/>
+        <limit lower="-${PI/2}" upper="${PI/2}" effort="100" velocity="1.0"/>
+    </joint>
+    <link name="2d_active_roll_link">
         <visual>
             <origin xyz="0 0 0" rpy="0 0 0"/>
@@ -111,5 +153,5 @@
                 <box size="${d_2djnt_a_L} ${d_2djnt_a_W} ${d_2djnt_a_H}"/>
             </geometry>
-            <material name="black"/>
+            <material name="red"/>
         </visual>
         <collision>
@@ -121,37 +163,7 @@
         <xacro:box_inertia m="${m_2djnt_a}" x="${d_2djnt_a_L}" y="${d_2djnt_a_W}" z="${d_2djnt_a_H}"/>
     </link>
-    <joint name="base_to_2d_active" type="fixed">
-        <parent link="base_link"/>
-        <child link="2d_active_link"/>
-        <origin xyz="0 0 -${d_2djnt_a_H/2}" rpy="0 0 0"/>
-    </joint>
-    ---
-    <link name="2d_passive_pitch_link"/>
-    <joint name="2d_pitch_joint" type="revolute">
-        <parent link="2d_active_link"/>
-        <child link="2d_passive_pitch_link"/>
-        <origin xyz="${-d_2djnt_a_L/2 - 0.059 + d_2djnt_p_L/2} 0 ${d_2djnt_a_H/2 - 0.080 - d_2djnt_p_H/2}" rpy="0 0 0"/>
-        <axis xyz="0 1 0"/>
-        <limit lower="-${PI/2}" upper="${PI/2}" effort="100" velocity="1.0"/>
-    </joint>
-    <link name="2d_passive_link">
-        <visual>
-            <origin xyz="0 0 0" rpy="0 0 0"/>
-            <geometry>
-                <box size="${d_2djnt_p_L} ${d_2djnt_p_W} ${d_2djnt_p_H}"/>
-            </geometry>
-            <material name="red"/>
-        </visual>
-        <collision>
-            <origin xyz="0 0 0" rpy="0 0 0"/>
-            <geometry>
-                <box size="${d_2djnt_p_L} ${d_2djnt_p_W} ${d_2djnt_p_H}"/>
-            </geometry>
-        </collision>
-        <xacro:box_inertia m="${m_2djnt}" x="${d_2djnt_p_L}" y="${d_2djnt_p_W}" z="${d_2djnt_p_H}"/>
-    </link>
     <joint name="2d_roll_joint" type="revolute">
-        <parent link="2d_passive_pitch_link"/>
-        <child link="2d_passive_link"/>
+        <parent link="2d_active_pitch_link"/>
+        <child link="2d_active_roll_link"/>
         <origin xyz="0 0 0" rpy="0 0 0"/>
         <axis xyz="1 0 0"/>
@@ -159,4 +171,5 @@
     </joint>
     ---
+    <!-- 2-DoF-to-Arm Connector -->
     <link name="2d_arm_connector_link">
         <visual>
@@ -176,9 +189,10 @@
     </link>
     <joint name="2d_passive_to_2d_arm_connector" type="fixed">
-        <parent link="2d_passive_link"/>
+        <parent link="2d_active_roll_link"/>
         <child link="2d_arm_connector_link"/>
-        <origin xyz="${(d_2djnt_p_L/2 - 0.022) + d_conn_L/2} 0 ${d_2djnt_p_H/2 - 0.0225 - d_conn_H/2}" rpy="0 0 0"/>
-    </joint>
-    ---
+        <origin xyz="${(d_2djnt_a_L/2 - 0.022) + d_conn_L/2} 0 ${d_2djnt_a_H/2 - 0.0225 - d_conn_H/2}" rpy="0 0 0"/>
+    </joint>
+    ---
+    <!-- Arm Segment #1 -->
     <xacro:arm_link_macro name="L1_link"/>
     <joint name="2d_arm_connector_to_L1" type="fixed">
@@ -196,4 +210,5 @@
     </joint>
     ---
+    <!-- Arm Segment #2 -->
     <xacro:arm_link_macro name="L2_link"/>
     <joint name="J1_to_L2" type="fixed">
@@ -211,4 +226,5 @@
     </joint>
     ---
+    <!-- Arm Segment #3 -->
     <xacro:arm_link_macro name="L3_link"/>
     <joint name="J2_to_L3" type="fixed">
@@ -226,4 +242,5 @@
     </joint>
     ---
+    <!-- Arm Segment #4 -->
     <xacro:arm_link_macro name="L4_link"/>
     <joint name="J3_to_L4" type="fixed">
@@ -246,5 +263,5 @@
             </geometry>
         </collision>
-        <xacro:box_inertia m="${m_manip_mount}" x="${d_arm_tip_L}" y="${d_arm_tip_W}" z="${d_arm_tip_H}"/>
+        <xacro:box_inertia m="${m_arm_tip}" x="${d_arm_tip_L}" y="${d_arm_tip_W}" z="${d_arm_tip_H}"/>
     </link>
     <joint name="L4_to_arm_tip" type="fixed">
@@ -254,18 +271,19 @@
     </joint>
     ---
+    <!-- Manipulator Joints -->
     <link name="mj1_link">
         <visual>
             <geometry>
-                <box size="${d_mj1_L} ${d_mj1_W} ${d_mj1_H}"/>
+                <box size="${d_MJ1_L} ${d_MJ1_W} ${d_MJ1_H}"/>
             </geometry>
             <material name="purple"/>
         </visual>
-        <collision><geometry><box size="${d_mj1_L} ${d_mj1_W} ${d_mj1_H}"/></geometry></collision>
-        <xacro:box_inertia m="${m_mj}" x="${d_mj1_L}" y="${d_mj1_W}" z="${d_mj1_H}"/>
-    </link>
-    <joint name="arm_tip_to_mj1" type="revolute">
+        <collision><geometry><box size="${d_MJ1_L} ${d_MJ1_W} ${d_MJ1_H}"/></geometry></collision>
+        <xacro:box_inertia m="${m_MJ}" x="${d_MJ1_L}" y="${d_MJ1_W}" z="${d_MJ1_H}"/>
+    </link>
+    <joint name="arm_tip_to_MJ1" type="revolute">
         <parent link="arm_tip_link"/>
         <child link="mj1_link"/>
-        <origin xyz="${(d_arm_tip_L/2 - 0.00875) - d_mj1_L/2} ${-d_arm_tip_W/2 - 0.0121 + d_mj1_W/2} ${(d_arm_tip_H/2 - 0.006) - d_mj1_H/2}" rpy="0 0 0"/>
+        <origin xyz="${(d_arm_tip_L/2 - 0.00875) - d_MJ1_L/2} ${-d_arm_tip_W/2 - 0.0121 + d_MJ1_W/2} ${(d_arm_tip_H/2 - 0.006) - d_MJ1_H/2}" rpy="0 0 0"/>
         <axis xyz="0 1 0"/>
         <limit lower="-${PI/2}" upper="${PI/2}" effort="50" velocity="1.5"/>
@@ -274,15 +292,15 @@
         <visual>
             <geometry>
-                <box size="${d_mj23_L} ${d_mj23_W} ${d_mj23_H}"/>
+                <box size="${d_MJ23_L} ${d_MJ23_W} ${d_MJ23_H}"/>
             </geometry>
             <material name="purple"/>
         </visual>
-        <collision><geometry><box size="${d_mj23_L} ${d_mj23_W} ${d_mj23_H}"/></geometry></collision>
-        <xacro:box_inertia m="${m_mj}" x="${d_mj23_L}" y="${d_mj23_W}" z="${d_mj23_H}"/>
-    </link>
-    <joint name="mj1_to_mj2" type="revolute">
+        <collision><geometry><box size="${d_MJ23_L} ${d_MJ23_W} ${d_MJ23_H}"/></geometry></collision>
+        <xacro:box_inertia m="${m_MJ}" x="${d_MJ23_L}" y="${d_MJ23_W}" z="${d_MJ23_H}"/>
+    </link>
+    <joint name="mj1_to_MJ2" type="revolute">
         <parent link="mj1_link"/>
         <child link="mj2_link"/>
-        <origin xyz="${(d_mj1_L/2 + 0.0295) - d_mj23_L/2} ${-d_mj1_W/2 - d_mj23_W/2} ${(d_mj1_H/2 + 0.0091) - d_mj23_H/2}" rpy="0 0 0"/>
+        <origin xyz="${(d_MJ1_L/2 + 0.0295) - d_MJ23_L/2} ${-d_MJ1_W/2 - d_MJ23_W/2} ${(d_MJ1_H/2 + 0.0091) - d_MJ23_H/2}" rpy="0 0 0"/>
         <axis xyz="0 0 1"/>
         <limit lower="-${PI/2}" upper="${PI/2}" effort="50" velocity="1.5"/>
@@ -291,20 +309,21 @@
         <visual>
             <geometry>
-                <box size="${d_mj23_L} ${d_mj23_H} ${d_mj23_W}"/>
+                <box size="${d_MJ23_L} ${d_MJ23_H} ${d_MJ23_W}"/>
             </geometry>
             <material name="purple"/>
         </visual>
-        <collision><geometry><box size="${d_mj23_L} ${d_mj23_H} ${d_mj23_W}"/></geometry></collision>
-        <xacro:box_inertia m="${m_mj}" x="${d_mj23_L}" y="${d_mj23_H}" z="${d_mj23_W}"/>
-    </link>
-    <joint name="mj2_to_mj3" type="revolute">
+        <collision><geometry><box size="${d_MJ23_L} ${d_MJ23_H} ${d_MJ23_W}"/></geometry></collision>
+        <xacro:box_inertia m="${m_MJ}" x="${d_MJ23_L}" y="${d_MJ23_H}" z="${d_MJ23_W}"/>
+    </link>
+    <joint name="mj2_to_MJ3" type="revolute">
         <parent link="mj2_link"/>
         <child link="mj3_link"/>
-        <origin xyz="${(-d_mj23_L/2 + 0.00025) + d_mj23_L/2} ${d_mj23_W/2 + 0.0053 - d_mj23_H/2} ${d_mj23_H/2 + d_mj23_W/2}" rpy="0 0 0"/>
+        <origin xyz="${(-d_MJ23_L/2 + 0.00025) + d_MJ23_L/2} ${d_MJ23_W/2 + 0.0053 - d_MJ23_H/2} ${d_MJ23_H/2 + d_MJ23_W/2}" rpy="0 0 0"/>
         <axis xyz="0 1 0"/>
         <limit lower="-${PI/2}" upper="${PI/2}" effort="50" velocity="1.5"/>
     </joint>
-    <gazebo reference="2d_active_link"><material>Gazebo/Black</material></gazebo>
-    <gazebo reference="2d_passive_link"><material>Gazebo/Red</material></gazebo>
+    <!-- ********************[ GAZEBO CONFIG ]******************** -->
+    <gazebo reference="2d_passive_link"><material>Gazebo/Black</material></gazebo>
+    <gazebo reference="2d_active_roll_link"><material>Gazebo/Red</material></gazebo>
     <gazebo reference="2d_arm_connector_link"><material>Gazebo/Black</material></gazebo>
     <gazebo reference="L1_link"><material>Gazebo/Gray</material></gazebo>

Commit message: added and aligned 2-DoF meshes

File: ros2_ws/src/libra/models/2dof_and_arm.urdf.xacro (robot description, xacro)
@@ -17,6 +17,6 @@
     <xacro:property name="d_conn_L" value="0.076"/>
     <xacro:property name="d_conn_W" value="0.076"/>
-    <xacro:property name="d_conn_H" value="0.076"/>
-    <xacro:property name="m_conn" value="0.187"/>
+    <xacro:property name="d_conn_H" value="0.0985"/>
+    <xacro:property name="m_conn" value="0.326"/>
     <!-- Arm Links -->
     <xacro:property name="d_L_len" value="0.900"/>
@@ -118,7 +118,7 @@
     <link name="2d_passive_link">
         <visual>
-            <origin xyz="0 0 0" rpy="0 0 0"/>
-            <geometry>
-                <box size="${d_2djnt_p_L} ${d_2djnt_p_W} ${d_2djnt_p_H}"/>
+            <origin xyz="-0.029 0 -0.042" rpy="${PI/2} 0 ${PI/2}"/>
+            <geometry>
+                <mesh filename="package://libra/meshes/2d-passive.stl" scale="0.001 0.001 0.001"/>
             </geometry>
             <material name="black"/>
@@ -149,7 +149,7 @@
     <link name="2d_active_roll_link">
         <visual>
-            <origin xyz="0 0 0" rpy="0 0 0"/>
-            <geometry>
-                <box size="${d_2djnt_a_L} ${d_2djnt_a_W} ${d_2djnt_a_H}"/>
+            <origin xyz="0 0 0.0050" rpy="-${PI/2} ${PI} -${PI/2}"/>
+            <geometry>
+                <mesh filename="package://libra/meshes/2d-active.stl" scale="0.001 0.001 0.001"/>
             </geometry>
             <material name="red"/>
@@ -174,7 +174,7 @@
     <link name="2d_arm_connector_link">
         <visual>
-            <origin xyz="0 0 0" rpy="0 0 0"/>
-            <geometry>
-                <box size="${d_conn_L} ${d_conn_W} ${d_conn_H}"/>
+            <origin xyz="0.0030 0 0.0267" rpy="${PI} 0 0"/>
+            <geometry>
+                <mesh filename="package://libra/meshes/2d-arm_connector.stl" scale="0.001 0.001 0.001"/>
             </geometry>
             <material name="black"/>
@@ -191,5 +191,5 @@
         <parent link="2d_active_roll_link"/>
         <child link="2d_arm_connector_link"/>
-        <origin xyz="${(d_2djnt_a_L/2 - 0.022) + d_conn_L/2} 0 ${d_2djnt_a_H/2 - 0.0225 - d_conn_H/2}" rpy="0 0 0"/>
+        <origin xyz="${(d_2djnt_a_L/2 - 0.022) + d_conn_L/2} 0 ${d_2djnt_a_H/2 - 0.020 - d_conn_H/2}" rpy="0 0 0"/>
     </joint>
     ---
@@ -199,5 +199,5 @@
         <parent link="2d_arm_connector_link"/>
         <child link="L1_link"/>
-        <origin xyz="${d_conn_L/2 + d_L_len/2} 0 0" rpy="0 0 0"/>
+        <origin xyz="${d_conn_L/2 + d_L_len/2} 0 -${d_conn_H/2 - 0.038}" rpy="0 0 0"/>
     </joint>
     <xacro:arm_joint_macro name="J1_link" L="${d_J12_L}" W="${d_J12_W}" H="${d_J12_H}" mass="${m_J12}"/>

Commit message: added mesh todos

File: ros2_ws/src/libra/models/2dof_and_arm.urdf.xacro (robot description, xacro)
@@ -81,4 +81,7 @@
                 <geometry>
                     <cylinder length="${d_L_len}" radius="${d_L_rad}"/>
+                    <!-- TODO
+                    <mesh filename="package://libra/meshes/arm-link.stl" scale="0.001 0.001 0.001"/>
+                    -->
                 </geometry>
                 <material name="gray"/>
@@ -99,4 +102,8 @@
                 <geometry>
                     <box size="${L} ${W} ${H}"/>
+                    <!-- TODO
+                    <mesh filename="package://libra/meshes/arm-j1_2.stl" scale="0.001 0.001 0.001"/>
+                    <mesh filename="package://libra/meshes/arm-j3.stl" scale="0.001 0.001 0.001"/>
+                    -->
                 </geometry>
                 <material name="red"/>
@@ -254,4 +261,7 @@
             <geometry>
                 <box size="${d_arm_tip_L} ${d_arm_tip_W} ${d_arm_tip_H}"/>
+                <!-- TODO
+                <mesh filename="package://libra/meshes/arm-tip.stl" scale="0.001 0.001 0.001"/>
+                -->
             </geometry>
             <material name="black"/>
@@ -274,6 +284,10 @@
     <link name="mj1_link">
         <visual>
+            <origin xyz="0 0 0" rpy="0 0 0"/>
             <geometry>
                 <box size="${d_MJ1_L} ${d_MJ1_W} ${d_MJ1_H}"/>
+                <!-- TODO
+                <mesh filename="package://libra/meshes/manip-j1.stl" scale="0.001 0.001 0.001"/>
+                -->
             </geometry>
             <material name="purple"/>
@@ -291,6 +305,10 @@
     <link name="mj2_link">
         <visual>
+            <origin xyz="0 0 0" rpy="0 0 0"/>
             <geometry>
                 <box size="${d_MJ23_L} ${d_MJ23_W} ${d_MJ23_H}"/>
+                <!-- TODO
+                <mesh filename="package://libra/meshes/manip-j2_3.stl" scale="0.001 0.001 0.001"/>
+                -->
             </geometry>
             <material name="purple"/>
@@ -308,6 +326,10 @@
     <link name="mj3_link">
         <visual>
+            <origin xyz="0 0 0" rpy="0 0 0"/>
             <geometry>
                 <box size="${d_MJ23_L} ${d_MJ23_H} ${d_MJ23_W}"/>
+                <!-- TODO
+                <mesh filename="package://libra/meshes/manip-j2_3.stl" scale="0.001 0.001 0.001"/>
+                -->
             </geometry>
             <material name="purple"/>
