Commit message: grouping like blocks and renaming link for better readability

File: ros2_ws/src/libra/models/2dof_and_arm.urdf.xacro (robot description, xacro)
@@ -20,7 +20,7 @@
     <xacro:property name="m_conn" value="0.326"/>
     <!-- Arm Links -->
-    <xacro:property name="d_L_len" value="0.900"/>
-    <xacro:property name="d_L_rad" value="0.030"/>
-    <xacro:property name="m_L" value="0.395"/>
+    <xacro:property name="d_arm_link_L" value="0.900"/>
+    <xacro:property name="d_arm_link_R" value="0.030"/>
+    <xacro:property name="m_arm_link" value="0.395"/>
     <!-- Arm Joints -->
     <xacro:property name="d_J12_L" value="0.12914"/>
@@ -80,5 +80,5 @@
                 <origin xyz="0 0 0" rpy="0 ${PI/2} 0"/>
                 <geometry>
-                    <cylinder length="${d_L_len}" radius="${d_L_rad}"/>
+                    <cylinder length="${d_arm_link_L}" radius="${d_arm_link_R}"/>
                     <!-- TODO
                     <mesh filename="package://libra/meshes/arm-link.stl" scale="0.001 0.001 0.001"/>
@@ -90,8 +90,8 @@
                 <origin xyz="0 0 0" rpy="0 ${PI/2} 0"/>
                 <geometry>
-                    <cylinder length="${d_L_len}" radius="${d_L_rad}"/>
+                    <cylinder length="${d_arm_link_L}" radius="${d_arm_link_R}"/>
                 </geometry>
             </collision>
-            <xacro:cylinder_inertia m="${m_L}" r="${d_L_rad}" h="${d_L_len}"/>
+            <xacro:cylinder_inertia m="${m_arm_link}" r="${d_arm_link_R}" h="${d_arm_link_L}"/>
         </link>
     </xacro:macro>
@@ -206,5 +206,5 @@
         <parent link="2d_arm_connector_link"/>
         <child link="L1_link"/>
-        <origin xyz="${d_conn_L/2 + d_L_len/2} 0 -${d_conn_H/2 - 0.038}" rpy="0 0 0"/>
+        <origin xyz="${d_conn_L/2 + d_arm_link_L/2} 0 -${d_conn_H/2 - 0.038}" rpy="0 0 0"/>
     </joint>
     <xacro:arm_joint_macro name="J1_link" L="${d_J12_L}" W="${d_J12_W}" H="${d_J12_H}" mass="${m_J12}"/>
@@ -212,5 +212,5 @@
         <parent link="L1_link"/>
         <child link="J1_link"/>
-        <origin xyz="${d_L_len/2 + d_J12_L/2} 0 ${-0.038 + d_J12_H/2}" rpy="0 0 0"/>
+        <origin xyz="${d_arm_link_L/2 + d_J12_L/2} 0 ${-0.038 + d_J12_H/2}" rpy="0 0 0"/>
         <axis xyz="0 0 1"/>
         <limit lower="-${PI}" upper="${PI}" effort="100" velocity="1.0"/>
@@ -222,5 +222,5 @@
         <parent link="J1_link"/>
         <child link="L2_link"/>
-        <origin xyz="${(d_J12_L/2 - 0.04014) + d_L_len/2} 0 ${d_J12_H/2 - 0.038}" rpy="0 0 0"/>
+        <origin xyz="${(d_J12_L/2 - 0.04014) + d_arm_link_L/2} 0 ${d_J12_H/2 - 0.038}" rpy="0 0 0"/>
     </joint>
     <xacro:arm_joint_macro name="J2_link" L="${d_J12_L}" W="${d_J12_W}" H="${d_J12_H}" mass="${m_J12}"/>
@@ -228,5 +228,5 @@
         <parent link="L2_link"/>
         <child link="J2_link"/>
-        <origin xyz="${d_L_len/2 + d_J12_L/2} 0 ${0.038 - d_J12_H/2}" rpy="0 0 0"/>
+        <origin xyz="${d_arm_link_L/2 + d_J12_L/2} 0 ${0.038 - d_J12_H/2}" rpy="0 0 0"/>
         <axis xyz="0 0 1"/>
         <limit lower="-${PI}" upper="${PI}" effort="100" velocity="1.0"/>
@@ -238,5 +238,5 @@
         <parent link="J2_link"/>
         <child link="L3_link"/>
-        <origin xyz="${(d_J12_L/2 - 0.04014) + d_L_len/2} 0 ${-d_J12_H/2 + 0.038}" rpy="0 0 0"/>
+        <origin xyz="${(d_J12_L/2 - 0.04014) + d_arm_link_L/2} 0 ${-d_J12_H/2 + 0.038}" rpy="0 0 0"/>
     </joint>
     <xacro:arm_joint_macro name="J3_link" L="${d_J3_L}" W="${d_J3_W}" H="${d_J3_H}" mass="${m_J3}"/>
@@ -244,5 +244,5 @@
         <parent link="L3_link"/>
         <child link="J3_link"/>
-        <origin xyz="${d_L_len/2 + d_J3_L/2} ${-0.03805 + d_J3_W/2} 0" rpy="0 0 0"/>
+        <origin xyz="${d_arm_link_L/2 + d_J3_L/2} ${-0.03805 + d_J3_W/2} 0" rpy="0 0 0"/>
         <axis xyz="0 1 0"/>
         <limit lower="-${PI/2}" upper="${PI/2}" effort="100" velocity="1.0"/>
@@ -254,5 +254,5 @@
         <parent link="J3_link"/>
         <child link="L4_link"/>
-        <origin xyz="${(d_J3_L/2 - 0.04014) + d_L_len/2} ${d_J3_W/2 - 0.038} 0" rpy="0 0 0"/>
+        <origin xyz="${(d_J3_L/2 - 0.04014) + d_arm_link_L/2} ${d_J3_W/2 - 0.038} 0" rpy="0 0 0"/>
     </joint>
     <link name="arm_tip_link">
@@ -278,5 +278,5 @@
         <parent link="L4_link"/>
         <child link="arm_tip_link"/>
-        <origin xyz="${d_L_len/2 + d_arm_tip_L/2} 0 ${0.042 - d_arm_tip_H/2}" rpy="0 0 0"/>
+        <origin xyz="${d_arm_link_L/2 + d_arm_tip_L/2} 0 ${0.042 - d_arm_tip_H/2}" rpy="0 0 0"/>
     </joint>
     ---
@@ -293,5 +293,10 @@
             <material name="purple"/>
         </visual>
-        <collision><geometry><box size="${d_MJ1_L} ${d_MJ1_W} ${d_MJ1_H}"/></geometry></collision>
+        <collision>
+            <origin xyz="0 0 0" rpy="0 0 0"/>
+            <geometry>
+                <box size="${d_MJ1_L} ${d_MJ1_W} ${d_MJ1_H}"/>
+            </geometry>
+        </collision>
         <xacro:box_inertia m="${m_MJ}" x="${d_MJ1_L}" y="${d_MJ1_W}" z="${d_MJ1_H}"/>
     </link>
@@ -314,5 +319,10 @@
             <material name="purple"/>
         </visual>
-        <collision><geometry><box size="${d_MJ23_L} ${d_MJ23_W} ${d_MJ23_H}"/></geometry></collision>
+        <collision>
+            <origin xyz="0 0 0" rpy="0 0 0"/>
+            <geometry>
+                <box size="${d_MJ23_L} ${d_MJ23_W} ${d_MJ23_H}"/>
+            </geometry>
+        </collision>
         <xacro:box_inertia m="${m_MJ}" x="${d_MJ23_L}" y="${d_MJ23_W}" z="${d_MJ23_H}"/>
     </link>
@@ -335,5 +345,10 @@
             <material name="purple"/>
         </visual>
-        <collision><geometry><box size="${d_MJ23_L} ${d_MJ23_H} ${d_MJ23_W}"/></geometry></collision>
+        <collision>
+            <origin xyz="0 0 0" rpy="0 0 0"/>
+            <geometry>
+                <box size="${d_MJ23_L} ${d_MJ23_H} ${d_MJ23_W}"/>
+            </geometry>
+        </collision>
         <xacro:box_inertia m="${m_MJ}" x="${d_MJ23_L}" y="${d_MJ23_H}" z="${d_MJ23_W}"/>
     </link>

Commit message: use actual convention for naming...

File: ros2_ws/src/libra/models/2dof_and_arm.urdf.xacro (robot description, xacro)
@@ -4,14 +4,14 @@
     <!-- Common -->
     <xacro:property name="PI" value="3.14159265359"/>
-    <!-- 2-DoF Joint (static part - "passive") -->
-    <xacro:property name="d_2djnt_p_L" value="0.143"/>
-    <xacro:property name="d_2djnt_p_W" value="0.165"/>
-    <xacro:property name="d_2djnt_p_H" value="0.1565"/>
-    <xacro:property name="m_2djnt_p" value="2.056"/>
-    <!-- 2-DoF Joint (moved part - "active") -->
-    <xacro:property name="d_2djnt_a_L" value="0.204"/>
-    <xacro:property name="d_2djnt_a_W" value="0.145"/>
-    <xacro:property name="d_2djnt_a_H" value="0.090"/>
-    <xacro:property name="m_2djnt_a" value="1.317"/>
+    <!-- 2-DoF Joint (static part - "stator") -->
+    <xacro:property name="d_2djnt_s_L" value="0.143"/>
+    <xacro:property name="d_2djnt_s_W" value="0.165"/>
+    <xacro:property name="d_2djnt_s_H" value="0.1565"/>
+    <xacro:property name="m_2djnt_s" value="2.056"/>
+    <!-- 2-DoF Joint (moved part - "rotor") -->
+    <xacro:property name="d_2djnt_r_L" value="0.204"/>
+    <xacro:property name="d_2djnt_r_W" value="0.145"/>
+    <xacro:property name="d_2djnt_r_H" value="0.090"/>
+    <xacro:property name="m_2djnt_r" value="1.317"/>
     <!-- 2-DoF-to-Arm Connector -->
     <xacro:property name="d_conn_L" value="0.076"/>
@@ -122,10 +122,10 @@
     <link name="base_link"/>
     ---
-    <!-- 2-DoF Joint (passive part) -->
-    <link name="2d_passive_link">
+    <!-- 2-DoF Joint (stator half) -->
+    <link name="2d_stator_link">
         <visual>
             <origin xyz="-0.029 0 -0.042" rpy="${PI/2} 0 ${PI/2}"/>
             <geometry>
-                <mesh filename="package://libra/meshes/2d-passive.stl" scale="0.001 0.001 0.001"/>
+                <mesh filename="package://libra/meshes/2d-stator.stl" scale="0.001 0.001 0.001"/>
             </geometry>
             <material name="black"/>
@@ -134,29 +134,29 @@
             <origin xyz="0 0 0" rpy="0 0 0"/>
             <geometry>
-                <box size="${d_2djnt_p_L} ${d_2djnt_p_W} ${d_2djnt_p_H}"/>
-            </geometry>
-        </collision>
-        <xacro:box_inertia m="${m_2djnt_p}" x="${d_2djnt_p_L}" y="${d_2djnt_p_W}" z="${d_2djnt_p_H}"/>
+                <box size="${d_2djnt_s_L} ${d_2djnt_s_W} ${d_2djnt_s_H}"/>
+            </geometry>
+        </collision>
+        <xacro:box_inertia m="${m_2djnt_s}" x="${d_2djnt_s_L}" y="${d_2djnt_s_W}" z="${d_2djnt_s_H}"/>
     </link>
     <joint name="base_to_2d" type="fixed">
         <parent link="base_link"/>
-        <child link="2d_passive_link"/>
-        <origin xyz="0 0 -${d_2djnt_p_H/2}" rpy="0 0 0"/>
-    </joint>
-    ---
-    <!-- 2-DoF Joint (active part) -->
-    <link name="2d_active_pitch_link"/>
+        <child link="2d_stator_link"/>
+        <origin xyz="0 0 -${d_2djnt_s_H/2}" rpy="0 0 0"/>
+    </joint>
+    ---
+    <!-- 2-DoF Joint (rotor half) -->
+    <link name="2d_rotor_pitch_link"/>
     <joint name="2d_pitch_joint" type="revolute">
-        <parent link="2d_passive_link"/>
-        <child link="2d_active_pitch_link"/>
-        <origin xyz="${-d_2djnt_p_L/2 - 0.059 + d_2djnt_a_L/2} 0 ${d_2djnt_p_H/2 - 0.080 - d_2djnt_a_H/2}" rpy="0 0 0"/>
+        <parent link="2d_stator_link"/>
+        <child link="2d_rotor_pitch_link"/>
+        <origin xyz="${-d_2djnt_s_L/2 - 0.059 + d_2djnt_r_L/2} 0 ${d_2djnt_s_H/2 - 0.080 - d_2djnt_r_H/2}" rpy="0 0 0"/>
         <axis xyz="0 1 0"/>
         <limit lower="-${PI/2}" upper="${PI/2}" effort="100" velocity="1.0"/>
     </joint>
-    <link name="2d_active_roll_link">
+    <link name="2d_rotor_roll_link">
         <visual>
             <origin xyz="0 0 0.0050" rpy="-${PI/2} ${PI} -${PI/2}"/>
             <geometry>
-                <mesh filename="package://libra/meshes/2d-active.stl" scale="0.001 0.001 0.001"/>
+                <mesh filename="package://libra/meshes/2d-rotor.stl" scale="0.001 0.001 0.001"/>
             </geometry>
             <material name="red"/>
@@ -165,12 +165,12 @@
             <origin xyz="0 0 0" rpy="0 0 0"/>
             <geometry>
-                <box size="${d_2djnt_a_L} ${d_2djnt_a_W} ${d_2djnt_a_H}"/>
-            </geometry>
-        </collision>
-        <xacro:box_inertia m="${m_2djnt_a}" x="${d_2djnt_a_L}" y="${d_2djnt_a_W}" z="${d_2djnt_a_H}"/>
+                <box size="${d_2djnt_r_L} ${d_2djnt_r_W} ${d_2djnt_r_H}"/>
+            </geometry>
+        </collision>
+        <xacro:box_inertia m="${m_2djnt_r}" x="${d_2djnt_r_L}" y="${d_2djnt_r_W}" z="${d_2djnt_r_H}"/>
     </link>
     <joint name="2d_roll_joint" type="revolute">
-        <parent link="2d_active_pitch_link"/>
-        <child link="2d_active_roll_link"/>
+        <parent link="2d_rotor_pitch_link"/>
+        <child link="2d_rotor_roll_link"/>
         <origin xyz="0 0 0" rpy="0 0 0"/>
         <axis xyz="1 0 0"/>
@@ -195,8 +195,8 @@
         <xacro:box_inertia m="${m_conn}" x="${d_conn_L}" y="${d_conn_W}" z="${d_conn_H}"/>
     </link>
-    <joint name="2d_passive_to_2d_arm_connector" type="fixed">
-        <parent link="2d_active_roll_link"/>
+    <joint name="2d_stator_to_2d_arm_connector" type="fixed">
+        <parent link="2d_rotor_roll_link"/>
         <child link="2d_arm_connector_link"/>
-        <origin xyz="${(d_2djnt_a_L/2 - 0.022) + d_conn_L/2} 0 ${d_2djnt_a_H/2 - 0.020 - d_conn_H/2}" rpy="0 0 0"/>
+        <origin xyz="${(d_2djnt_r_L/2 - 0.022) + d_conn_L/2} 0 ${d_2djnt_r_H/2 - 0.020 - d_conn_H/2}" rpy="0 0 0"/>
     </joint>
     ---
@@ -361,6 +361,6 @@
     </joint>
     <!-- ********************[ GAZEBO CONFIG ]******************** -->
-    <gazebo reference="2d_passive_link"><material>Gazebo/Black</material></gazebo>
-    <gazebo reference="2d_active_roll_link"><material>Gazebo/Red</material></gazebo>
+    <gazebo reference="2d_stator_link"><material>Gazebo/Black</material></gazebo>
+    <gazebo reference="2d_rotor_roll_link"><material>Gazebo/Red</material></gazebo>
     <gazebo reference="2d_arm_connector_link"><material>Gazebo/Black</material></gazebo>
     <gazebo reference="L1_link"><material>Gazebo/Gray</material></gazebo>

Commit message: add link meshes

File: ros2_ws/src/libra/models/2dof_and_arm.urdf.xacro (robot description, xacro)
@@ -78,10 +78,7 @@
         <link name="${name}">
             <visual>
-                <origin xyz="0 0 0" rpy="0 ${PI/2} 0"/>
+                <origin xyz="0 0 0" rpy="0 ${PI/2} ${PI/2}"/>
                 <geometry>
-                    <cylinder length="${d_arm_link_L}" radius="${d_arm_link_R}"/>
-                    <!-- TODO
                     <mesh filename="package://libra/meshes/arm-link.stl" scale="0.001 0.001 0.001"/>
-                    -->
                 </geometry>
                 <material name="gray"/>

Commit message: minor capitalization fix

File: ros2_ws/src/libra/models/2dof_and_arm.urdf.xacro (robot description, xacro)
@@ -353,5 +353,5 @@
         <xacro:box_inertia m="${m_MJ}" x="${d_MJ23_L}" y="${d_MJ23_H}" z="${d_MJ23_W}"/>
     </link>
-    <joint name="mj2_to_MJ3" type="revolute">
+    <joint name="mj2_to_mj3" type="revolute">
         <parent link="mj2_link"/>
         <child link="mj3_link"/>
