Commit message: rename for so it matches intuitiveness of upcoming commit

File: ros2_ws/src/libra/models/sensor_suite.urdf.xacro (robot description, xacro)
@@ -66,5 +66,5 @@
             <origin xyz="0 0 0" rpy="${PI/2} 0 ${PI/2}"/>
             <geometry>
-                <mesh filename="package://libra/meshes/M02-1_Sensor-Mount_LIDAR_guard.stl" scale="0.001 0.001 0.001"/>
+                <mesh filename="package://libra/meshes/mount_g-lidar.stl" scale="0.001 0.001 0.001"/>
             </geometry>
             <material name="black"/>
@@ -86,5 +86,5 @@
             <origin xyz="0.013602 0 0.028351" rpy="0 0 -${PI/2}"/>
             <geometry>
-                <mesh filename="package://libra/meshes/SF45-B_simplified.stl" scale="0.001 0.001 0.001"/>
+                <mesh filename="package://libra/meshes/lidar_sf45b-simplified.stl" scale="0.001 0.001 0.001"/>
             </geometry>
             <material name="purple"/>
@@ -106,5 +106,5 @@
             <origin xyz="0 0 0" rpy="-${PI/2} 0 ${PI/2}"/>
             <geometry>
-                <mesh filename="package://libra/meshes/M02-0_Sensor-Mount_Camera_guard.stl" scale="0.001 0.001 0.001"/>
+                <mesh filename="package://libra/meshes/mount_g-realsense.stl" scale="0.001 0.001 0.001"/>
             </geometry>
             <material name="black"/>
@@ -126,5 +126,5 @@
             <origin xyz="0.026 0 0" rpy="${PI/2} 0 ${PI/2}"/>
             <geometry>
-                <mesh filename="package://libra/meshes/D456.stl" scale="0.001 0.001 0.001"/>
+                <mesh filename="package://libra/meshes/realsense_d456.stl" scale="0.001 0.001 0.001"/>
             </geometry>
             <material name="silver"/>

Commit message: standardize naming

File: ros2_ws/src/libra/models/sensor_suite.urdf.xacro (robot description, xacro)
@@ -3,24 +3,24 @@
     <!-- ********************[ PROPERTIES ]******************** -->
     <!-- Common -->
-    <xacro:property name="PI" value="3.14159"/>
+    <xacro:property name="PI" value="3.14159265359"/>
     <!-- Mounts -->
-    <xacro:property name="mount_lidar_width" value="0.100000"/>
-    <xacro:property name="mount_lidar_height" value="0.084000"/>
-    <xacro:property name="mount_lidar_depth" value="0.012514"/>
-    <xacro:property name="mount_lidar_mass" value="0.009"/>
-    <xacro:property name="mount_camera_width" value="0.135861"/>
-    <xacro:property name="mount_camera_height" value="0.059941"/>
-    <xacro:property name="mount_camera_depth" value="0.104349"/>
-    <xacro:property name="mount_camera_mass" value="0.056"/>
+    <xacro:property name="m_lidar_L" value="0.012514"/>
+    <xacro:property name="m_lidar_W" value="0.100000"/>
+    <xacro:property name="m_lidar_H" value="0.084000"/>
+    <xacro:property name="m_lidar_m" value="0.009"/>
+    <xacro:property name="m_camera_L" value="0.104349"/>
+    <xacro:property name="m_camera_W" value="0.135861"/>
+    <xacro:property name="m_camera_H" value="0.059941"/>
+    <xacro:property name="m_camera_m" value="0.056"/>
     <!-- Spinning 2D LIDAR (SF45-B, LightWare) -->
-    <xacro:property name="lidar_width" value="0.048462"/>
-    <xacro:property name="lidar_height" value="0.043979"/>
-    <xacro:property name="lidar_depth" value="0.050587"/>
-    <xacro:property name="lidar_mass" value="0.058"/>
+    <xacro:property name="lidar_W" value="0.048462"/>
+    <xacro:property name="lidar_H" value="0.043979"/>
+    <xacro:property name="lidar_L" value="0.050587"/>
+    <xacro:property name="lidar_m" value="0.058"/>
     <!-- RGB-D camera (RealSense D456, Intel) -->
-    <xacro:property name="camera_width" value="0.123999"/>
-    <xacro:property name="camera_height" value="0.029093"/>
-    <xacro:property name="camera_depth" value="0.026004"/>
-    <xacro:property name="camera_mass" value="0.116"/>
+    <xacro:property name="camera_W" value="0.123999"/>
+    <xacro:property name="camera_H" value="0.029093"/>
+    <xacro:property name="camera_L" value="0.026004"/>
+    <xacro:property name="camera_m" value="0.116"/>
     <!-- ********************[ MATERIALS ]******************** -->
     <material name="black">
@@ -73,11 +73,11 @@
             <origin xyz="0 0 0" rpy="0 0 0"/>
             <geometry>
-                <box size="${mount_lidar_depth} ${mount_lidar_width} ${mount_lidar_height}"/>
+                <box size="${m_lidar_L} ${m_lidar_W} ${m_lidar_H}"/>
             </geometry>
         </collision>
-        <xacro:box_inertia m="${mount_lidar_mass}"
-                           x="${mount_lidar_depth}"
-                           y="${mount_lidar_width}"
-                           z="${mount_lidar_height}"/>
+        <xacro:box_inertia m="${m_lidar_m}"
+                           x="${m_lidar_L}"
+                           y="${m_lidar_W}"
+                           z="${m_lidar_H}"/>
     </link>
     <!-- LIDAR -->
@@ -91,13 +91,13 @@
         </visual>
         <collision>
-            <origin xyz="0 0 ${lidar_height/2}" rpy="0 0 0"/>
+            <origin xyz="0 0 ${lidar_H/2}" rpy="0 0 0"/>
             <geometry>
-                <box size="${lidar_depth} ${lidar_width} ${lidar_height}"/>
+                <box size="${lidar_L} ${lidar_W} ${lidar_H}"/>
             </geometry>
         </collision>
-        <xacro:box_inertia m="${lidar_mass}"
-                           x="${lidar_depth}"
-                           y="${lidar_width}"
-                           z="${lidar_height}"/>
+        <xacro:box_inertia m="${lidar_m}"
+                           x="${lidar_L}"
+                           y="${lidar_W}"
+                           z="${lidar_H}"/>
     </link>
     <!-- Camera Mount -->
@@ -113,11 +113,11 @@
             <origin xyz="0.045175 0 0.009540" rpy="0 0 0"/>
             <geometry>
-                <box size="${mount_camera_depth} ${mount_camera_width} ${mount_camera_height}"/>
+                <box size="${m_camera_L} ${m_camera_W} ${m_camera_H}"/>
             </geometry>
         </collision>
-        <xacro:box_inertia m="${mount_camera_mass}"
-                           x="${mount_camera_depth}"
-                           y="${mount_camera_width}"
-                           z="${mount_camera_height}"/>
+        <xacro:box_inertia m="${m_camera_m}"
+                           x="${m_camera_L}"
+                           y="${m_camera_W}"
+                           z="${m_camera_H}"/>
     </link>
     <!-- Camera -->
@@ -131,13 +131,13 @@
         </visual>
         <collision>
-            <origin xyz="${camera_depth/2} 0 0" rpy="0 0 0"/>
+            <origin xyz="${camera_L/2} 0 0" rpy="0 0 0"/>
             <geometry>
-                <box size="${camera_depth} ${camera_width} ${camera_height}"/>
+                <box size="${camera_L} ${camera_W} ${camera_H}"/>
             </geometry>
         </collision>
-        <xacro:box_inertia m="${camera_mass}"
-                           x="${camera_depth}"
-                           y="${camera_width}"
-                           z="${camera_height}"/>
+        <xacro:box_inertia m="${camera_m}"
+                           x="${camera_L}"
+                           y="${camera_W}"
+                           z="${camera_H}"/>
     </link>
     <!-- ********************[ JOINTS ]******************** -->

Commit message: changed name of sensor suite base link in preparation for combination with new libra arm model

File: ros2_ws/src/libra/models/sensor_suite.urdf.xacro (robot description, xacro)
@@ -60,5 +60,5 @@
     <!-- ********************[ LINKS ]******************** -->
     <!-- Base Link -->
-    <link name="base_link"/>  <!-- sensor_suite_base -->
+    <link name="sensor_suite_base_link"/>
     <!-- LIDAR Mount -->
     <link name="mount_lidar_link">
@@ -144,5 +144,5 @@
     <!-- NOTE: X = forward/red, Y = left/green, Z = upwards/blue -->
     <joint name="base_to_mount_lidar" type="fixed">
-        <parent link="base_link"/>  <!-- sensor_suite_base -->
+        <parent link="sensor_suite_base_link"/>
         <child link="mount_lidar_link"/>
         <origin xyz="0.001 0 0" rpy="0 0 0"/>  <!-- accounts for mounting bracket -->
@@ -154,5 +154,5 @@
     </joint>
     <joint name="base_to_mount_camera" type="fixed">
-        <parent link="base_link"/>  <!-- sensor_suite_base -->
+        <parent link="sensor_suite_base_link"/>
         <child link="mount_camera_link"/>
         <origin xyz="-0.001 0 0" rpy="0 0 0"/>  <!-- accounts for mounting bracket -->
