Commit message: archived unneeded models

File: ros2_ws/src/libra/models/archive/2dof_and_arm.urdf.xacro (robot description, xacro)
@@ -15,7 +15,7 @@
     <xacro:property name="m_2djnt_r" value="1.317"/>
     <!-- 2-DoF-to-Arm Connector -->
-    <xacro:property name="d_conn_L" value="0.076"/>
-    <xacro:property name="d_conn_W" value="0.076"/>
-    <xacro:property name="d_conn_H" value="0.0985"/>
+    <xacro:property name="d_conn_arm_L" value="0.076"/>
+    <xacro:property name="d_conn_arm_W" value="0.076"/>
+    <xacro:property name="d_conn_arm_H" value="0.0985"/>
     <xacro:property name="m_conn" value="0.326"/>
     <!-- Arm Links -->
@@ -187,16 +187,16 @@
             <origin xyz="0 0 0" rpy="0 0 0"/>
             <geometry>
-                <box size="${d_conn_L} ${d_conn_W} ${d_conn_H}"/>
-            </geometry>
-        </collision>
-        <xacro:box_inertia m="${m_conn}" x="${d_conn_L}" y="${d_conn_W}" z="${d_conn_H}"/>
+                <box size="${d_conn_arm_L} ${d_conn_arm_W} ${d_conn_arm_H}"/>
+            </geometry>
+        </collision>
+        <xacro:box_inertia m="${m_conn}" x="${d_conn_arm_L}" y="${d_conn_arm_W}" z="${d_conn_arm_H}"/>
     </link>
     <joint name="2d_stator_to_2d_arm_connector" type="fixed">
         <parent link="2d_rotor_roll_link"/>
         <child link="2d_arm_connector_link"/>
-        <origin xyz="${(d_2djnt_r_L/2 - 0.022) + d_conn_L/2} 0 ${d_2djnt_r_H/2 - 0.020 - d_conn_H/2}" rpy="0 0 0"/>
-    </joint>
-    ---
-    <!-- TODO:
+        <origin xyz="${(d_2djnt_r_L/2 - 0.022) + d_conn_arm_L/2} 0 ${d_2djnt_r_H/2 - 0.020 - d_conn_arm_H/2}" rpy="0 0 0"/>
+    </joint>
+    ---
+    <!-- TODO
             Arm joints should be divided into stator/rotor pairs like the 2-DoF Joint.
     -->
@@ -206,5 +206,5 @@
         <parent link="2d_arm_connector_link"/>
         <child link="L1_link"/>
-        <origin xyz="${d_conn_L/2 + d_arm_link_L/2} 0 -${d_conn_H/2 - 0.038}" rpy="0 0 0"/>
+        <origin xyz="${d_conn_arm_L/2 + d_arm_link_L/2} 0 -${d_conn_arm_H/2 - 0.038}" rpy="0 0 0"/>
     </joint>
     <xacro:arm_joint_macro name="J1_link" L="${d_J12_L}" W="${d_J12_W}" H="${d_J12_H}" mass="${m_J12}"/>
