Commit message: use normalized outbound links

File: ros2_ws/src/libra/models/assemblies/sensor_suite.urdf.xacro (robot description, xacro)
@@ -40,5 +40,5 @@
             <parent link="${parent}"/>
             <child link="sensor_suite_base_link"/>
-            <origin xyz="0.03275 0 0" rpy="0 0 0"/>  <!-- dist. from MJ3 to mounting bracket end -->
+            <origin xyz="0 0 0" rpy="0 0 0"/>
         </joint>
         <!-- LIDAR Mount -->
@@ -62,5 +62,5 @@
             <parent link="sensor_suite_base_link"/>
             <child link="mount_lidar_link"/>
-            <origin xyz="0.001 0 0" rpy="0 0 0"/>  <!-- accounts for mounting bracket -->
+            <origin xyz="0.001 0 0" rpy="0 0 0"/>  <!-- accounts for mounting bracket thickness -->
         </joint>
         <!-- LIDAR -->
@@ -84,5 +84,5 @@
             <parent link="mount_lidar_link"/>
             <child link="lidar_link"/>
-            <origin xyz="0.006 0 0" rpy="0 ${PI/2} 0"/>  <!-- facing downwards-->
+            <origin xyz="0.006 0 0" rpy="0 ${PI/2} 0"/>  <!-- facing downwards -->
         </joint>
         ---
@@ -107,5 +107,5 @@
             <parent link="sensor_suite_base_link"/>
             <child link="mount_camera_link"/>
-            <origin xyz="-0.001 0 0" rpy="0 0 0"/>  <!-- accounts for mounting bracket -->
+            <origin xyz="-0.001 0 0" rpy="0 0 0"/>  <!-- accounts for mounting bracket thickness -->
         </joint>
         <!-- Camera -->

File: ros2_ws/src/libra/models/display_sensors.urdf.xacro (robot description, xacro)
@@ -7,5 +7,5 @@
 ****************************************************************************-->
 <robot name="Sensor_Suite" xmlns:xacro="http://www.ros.org/wiki/xacro">
-    <xacro:include filename="$(find libra)/models/assemblies/sensor_suite.urdf.xacro" />
+    <xacro:include filename="$(find libra)/models/assemblies/sensor_suite.urdf.xacro"/>
     <link name="base_link"/>
     <xacro:spawn_sensors parent="base_link"/>
