Commit message: added outbound link, standardized joint names, added limits

File: ros2_ws/src/libra/models/assemblies/2djnt.urdf.xacro (robot description, xacro)
@@ -44,5 +44,5 @@
             <xacro:box_inertia m="${m_2djnt_s}" x="${d_2djnt_s_L}" y="${d_2djnt_s_W}" z="${d_2djnt_s_H}"/>
         </link>
-        <joint name="${parent}_to_stator" type="fixed">
+        <joint name="${parent}_to_2d_stator" type="fixed">
             <parent link="${parent}"/>
             <child link="2d_stator_link"/>
@@ -57,5 +57,5 @@
             <origin xyz="${-d_2djnt_s_L/2 - 0.059 + d_2djnt_r_L/2} 0 ${d_2djnt_s_H/2 - 0.080 - d_2djnt_r_H/2}" rpy="0 0 0"/>
             <axis xyz="0 1 0"/>
-            <limit lower="-${PI/2}" upper="${PI/2}" effort="100" velocity="1.0"/>
+            <limit lower="${-10 * PI / 180.0}" upper="${90 * PI / 180.0}" effort="100" velocity="1.0"/>
         </joint>
         <link name="2d_rotor_roll_link">
@@ -76,9 +76,9 @@
             <origin xyz="0 0 0" rpy="0 0 0"/>
             <axis xyz="1 0 0"/>
-            <limit lower="-${PI/2}" upper="${PI/2}" effort="100" velocity="1.0"/>
+            <limit lower="${-10 * PI / 180.0}" upper="${10 * PI / 180.0}" effort="100" velocity="1.0"/>
         </joint>
         ---
         <!-- Arm Connector -->
-        <link name="2d_arm_connector_link">
+        <link name="arm_conn_link">
             <visual>
                 <origin xyz="0.0030 0 0.0267" rpy="${PI} 0 0"/>
@@ -92,13 +92,21 @@
             <xacro:box_inertia m="${m_conn_arm}" x="${d_conn_arm_L}" y="${d_conn_arm_W}" z="${d_conn_arm_H}"/>
         </link>
-        <joint name="rotor_to_connector" type="fixed">
+        <joint name="2d_roll_joint_to_2d_out_arm" type="fixed">
             <parent link="2d_rotor_roll_link"/>
-            <child link="2d_arm_connector_link"/>
+            <child link="arm_conn_link"/>
             <origin xyz="${(d_2djnt_r_L/2 - 0.022) + d_conn_arm_L/2} 0 ${d_2djnt_r_H/2 - 0.020 - d_conn_arm_H/2}" rpy="0 0 0"/>
+        </joint>
+        ---
+        <!-- Outbound Link -->
+        <link name="2d_out_arm_link"/>
+        <joint name="arm_conn_to_2d_out_arm" type="fixed">
+            <parent link="arm_conn_link"/>
+            <child link="2d_out_arm_link"/>
+            <origin xyz="${d_conn_arm_L/2} 0 -${d_conn_arm_H/2 - 0.038}" rpy="0 0 0"/>
         </joint>
         <!-- ********************[ GAZEBO CONFIG ]******************** -->
         <gazebo reference="2d_stator_link"><material>Gazebo/Black</material></gazebo>
         <gazebo reference="2d_rotor_roll_link"><material>Gazebo/Red</material></gazebo>
-        <gazebo reference="2d_arm_connector_link"><material>Gazebo/Black</material></gazebo>
+        <gazebo reference="arm_conn_link"><material>Gazebo/Black</material></gazebo>
     </xacro:macro>
 </robot>

File: ros2_ws/src/libra/models/display_2djnt.urdf.xacro (robot description, xacro)
@@ -7,5 +7,5 @@
 ****************************************************************************-->
 <robot name="LIBRA-I_2DJNT" xmlns:xacro="http://www.ros.org/wiki/xacro">
-    <xacro:include filename="$(find libra)/models/assemblies/2djnt.urdf.xacro" />
+    <xacro:include filename="$(find libra)/models/assemblies/2djnt.urdf.xacro"/>
     <link name="base_link"/>
     <xacro:spawn_2djnt parent="base_link"/>

Commit message: standardize name of 2djnt out link

File: ros2_ws/src/libra/models/assemblies/2djnt.urdf.xacro (robot description, xacro)
@@ -99,8 +99,8 @@
         ---
         <!-- Outbound Link -->
-        <link name="2d_out_arm_link"/>
+        <link name="2djnt_out_arm_link"/>
         <joint name="arm_conn_to_2d_out_arm" type="fixed">
             <parent link="arm_conn_link"/>
-            <child link="2d_out_arm_link"/>
+            <child link="2djnt_out_arm_link"/>
             <origin xyz="${d_conn_arm_L/2} 0 -${d_conn_arm_H/2 - 0.038}" rpy="0 0 0"/>
         </joint>

File: ros2_ws/src/libra/models/robots/libra1.urdf.xacro (robot description, xacro)
@@ -7,7 +7,8 @@
 ****************************************************************************-->
 <robot name="LIBRA-I" xmlns:xacro="http://www.ros.org/wiki/xacro">
-    <xacro:include filename="$(find libra)/models/assemblies/2djnt.urdf.xacro" />
-    <xacro:include filename="$(find libra)/models/assemblies/arm.urdf.xacro" />
-    <xacro:include filename="$(find libra)/models/assemblies/sensor_suite.urdf.xacro" />
+    <xacro:include filename="$(find libra)/models/assemblies/2djnt.urdf.xacro"/>
+    <xacro:include filename="$(find libra)/models/assemblies/arm.urdf.xacro"/>
+    <xacro:include filename="$(find libra)/models/assemblies/manip.urdf.xacro"/>
+    <xacro:include filename="$(find libra)/models/assemblies/sensor_suite.urdf.xacro"/>
     <!-- NOTE
         Black = static elements
@@ -19,5 +20,6 @@
     <link name="base_link"/>
     <xacro:spawn_2djnt parent="base_link"/>
-    <xacro:spawn_arm parent="2d_arm_connector_link"/>
-    <xacro:spawn_sensors parent="mj3_link"/>
+    <xacro:spawn_arm parent="2djnt_out_arm_link"/>
+    <xacro:spawn_manip parent="arm_out_link"/>
+    <xacro:spawn_sensors parent="manip_out_link"/>
 </robot>

File: ros2_ws/src/libra/models/robots/libra1_no_manip.urdf.xacro (robot description, xacro)
@@ -1,6 +1,6 @@
 <?xml version="1.0"?>
 <!--***************************************************************************
-/// @file   libra1_no_sensors.urdf.xacro
-/// @brief  LIBRA-I (sensorless) model constructor.
+/// @file   libra1_no_manip.urdf.xacro
+/// @brief  LIBRA-I (w/o customization) model constructor.
 ///
 /// @author brice.c.aa
@@ -17,4 +17,4 @@
     <link name="base_link"/>
     <xacro:spawn_2djnt parent="base_link"/>
-    <xacro:spawn_arm parent="2d_arm_connector_link"/>
+    <xacro:spawn_arm parent="2djnt_out_arm_link"/>
 </robot>

Commit message: rename joints

File: ros2_ws/src/libra/models/assemblies/2djnt.urdf.xacro (robot description, xacro)
@@ -52,5 +52,5 @@
         <!-- Rotor (moved part) -->
         <link name="2d_rotor_pitch_link"/>
-        <joint name="2d_pitch_joint" type="revolute">
+        <joint name="Pitch" type="revolute">
             <parent link="2d_stator_link"/>
             <child link="2d_rotor_pitch_link"/>
@@ -71,5 +71,5 @@
             <xacro:box_inertia m="${m_2djnt_r}" x="${d_2djnt_r_L}" y="${d_2djnt_r_W}" z="${d_2djnt_r_H}"/>
         </link>
-        <joint name="2d_roll_joint" type="revolute">
+        <joint name="Roll" type="revolute">
             <parent link="2d_rotor_pitch_link"/>
             <child link="2d_rotor_roll_link"/>
@@ -92,5 +92,5 @@
             <xacro:box_inertia m="${m_conn_arm}" x="${d_conn_arm_L}" y="${d_conn_arm_W}" z="${d_conn_arm_H}"/>
         </link>
-        <joint name="2d_roll_joint_to_2d_out_arm" type="fixed">
+        <joint name="2d_roll_to_2d_out_arm" type="fixed">
             <parent link="2d_rotor_roll_link"/>
             <child link="arm_conn_link"/>

File: ros2_ws/src/libra/models/assemblies/arm.urdf.xacro (robot description, xacro)
@@ -106,5 +106,5 @@
             </joint>
             <link name="${name}_hebi_rotor_link"/>
-            <joint name="${name}_hebi_stator_to_${name}_hebi_rotor" type="revolute">
+            <joint name="${name}" type="revolute">
                 <parent link="${name}_hebi_stator_link"/>
                 <child link="${name}_hebi_rotor_link"/>

File: ros2_ws/src/libra/models/assemblies/manip.urdf.xacro (robot description, xacro)
@@ -53,5 +53,5 @@
         </joint>
         <link name="MJ1_rotor_link"/>
-        <joint name="MJ1_stator_to_MJ1_rotor" type="revolute">
+        <joint name="MJ1" type="revolute">
             <parent link="MJ1_stator_link"/>
             <child link="MJ1_rotor_link"/>
@@ -84,5 +84,5 @@
         </joint>
         <link name="MJ2_rotor_link"/>
-        <joint name="MJ2_stator_to_MJ2_rotor" type="revolute">
+        <joint name="MJ2" type="revolute">
             <parent link="MJ2_stator_link"/>
             <child link="MJ2_rotor_link"/>
@@ -115,5 +115,5 @@
         </joint>
         <link name="MJ3_rotor_link"/>
-        <joint name="MJ3_stator_to_MJ3_rotor" type="revolute">
+        <joint name="MJ3" type="revolute">
             <parent link="MJ3_stator_link"/>
             <child link="MJ3_rotor_link"/>
