Commit message: added static manip, moved arm tip to manip

File: ros2_ws/src/libra/models/assemblies/arm.urdf.xacro (robot description, xacro)
@@ -34,9 +34,4 @@
         <xacro:property name="d_hebi_H" value="0.0451"/>
         <xacro:property name="m_hebi" value="0.490"/>
-        <!-- Arm Tip / Manipulator Mount -->
-        <xacro:property name="d_arm_tip_L" value="0.100"/>
-        <xacro:property name="d_arm_tip_W" value="0.070"/>
-        <xacro:property name="d_arm_tip_H" value="0.0935"/>
-        <xacro:property name="m_arm_tip" value="0.170"/>
         <!-- ********************[ MACROS ]******************** -->
         <xacro:macro name="link_macro" params="name">
@@ -198,31 +193,10 @@
             <origin xyz="${d_conn_inner_L/2 + d_arm_link_L/2} 0 0" rpy="${PI/2} 0 0"/>
         </joint>
-        <link name="arm_tip_link">
-            <visual>
-                <origin xyz="-${d_arm_tip_L/2} 0 ${d_arm_tip_H/2 - 0.002}" rpy="${PI/2} 0 ${PI/2}"/>
-                <geometry>
-                    <mesh filename="package://libra/meshes/arm-tip.stl" scale="0.001 0.001 0.001"/>
-                </geometry>
-                <material name="black"/>
-            </visual>
-            <collision>
-                <origin xyz="0 0 0" rpy="0 0 0"/>
-                <geometry>
-                    <box size="${d_arm_tip_L} ${d_arm_tip_W} ${d_arm_tip_H}"/>
-                </geometry>
-            </collision>
-            <xacro:box_inertia m="${m_arm_tip}" x="${d_arm_tip_L}" y="${d_arm_tip_W}" z="${d_arm_tip_H}"/>
-        </link>
-        <joint name="L4_to_arm_tip" type="fixed">
-            <parent link="L4_link"/>
-            <child link="arm_tip_link"/>
-            <origin xyz="${d_arm_link_L/2 + d_arm_tip_L/2} 0 ${0.042 - d_arm_tip_H/2}" rpy="0 0 0"/>
-        </joint>
         <!-- Outbound Link -->
         <link name="arm_out_link"/>
-        <joint name="arm_tip_to_arm_out" type="fixed">
-            <parent link="arm_tip_link"/>
+        <joint name="L4_to_arm_out" type="fixed">
+            <parent link="L4_link"/>
             <child link="arm_out_link"/>
-            <origin xyz="${d_arm_tip_L/2 - 0.029} ${-d_arm_tip_W/2} ${d_arm_tip_H/2 - 0.016}" rpy="0 0 0"/>
+            <origin xyz="${d_arm_link_L/2} 0 0" rpy="0 0 0"/>
         </joint>
         <!-- ********************[ GAZEBO CONFIG ]******************** -->
@@ -234,5 +208,4 @@
         <gazebo reference="J3_link"><material>Gazebo/Red</material></gazebo>
         <gazebo reference="L4_link"><material>Gazebo/Gray</material></gazebo>
-        <gazebo reference="arm_tip_link"><material>Gazebo/Black</material></gazebo>
     </xacro:macro>
 </robot>

File: ros2_ws/src/libra/models/assemblies/manip.urdf.xacro (robot description, xacro)
@@ -9,7 +9,12 @@
     <!-- Includes -->
     <xacro:include filename="$(find libra)/models/common/common.urdf.xacro" />
-    <!-- Definition -->
+    <!-- Definition #1: 3-Servo Manipulator -->
     <xacro:macro name="spawn_manip" params="parent">
         <!-- ********************[ PROPERTIES ]******************** -->
+        <!-- Servo Mount (arm tip) -->
+        <xacro:property name="d_servo_mount_L" value="0.100"/>
+        <xacro:property name="d_servo_mount_W" value="0.070"/>
+        <xacro:property name="d_servo_mount_H" value="0.0935"/>
+        <xacro:property name="m_servo_mount" value="0.170"/>
         <!-- Servo -->
         <xacro:property name="d_servo_L" value="0.054"/>
@@ -30,4 +35,26 @@
             X = forward/red, Y = left/green, Z = upwards/blue
         -->
+        <!-- Servo Mount (arm tip) -->
+        <link name="servo_mount_link">
+            <visual>
+                <origin xyz="-${d_servo_mount_L/2} 0 ${d_servo_mount_H/2 - 0.002}" rpy="${PI/2} 0 ${PI/2}"/>
+                <geometry>
+                    <mesh filename="package://libra/meshes/mount-servos.stl" scale="0.001 0.001 0.001"/>
+                </geometry>
+                <material name="black"/>
+            </visual>
+            <collision>
+                <origin xyz="0 0 0" rpy="0 0 0"/>
+                <geometry>
+                    <box size="${d_servo_mount_L} ${d_servo_mount_W} ${d_servo_mount_H}"/>
+                </geometry>
+            </collision>
+            <xacro:box_inertia m="${m_servo_mount}" x="${d_servo_mount_L}" y="${d_servo_mount_W}" z="${d_servo_mount_H}"/>
+        </link>
+        <joint name="parent_to_servo_mount" type="fixed">
+            <parent link="${parent}"/>
+            <child link="servo_mount_link"/>
+            <origin xyz="${d_servo_mount_L/2} 0 ${0.042 - d_servo_mount_H/2}" rpy="0 0 0"/>
+        </joint>
         <!-- Manipulator Joint #1 (servo) -->
         <link name="MJ1_stator_link">
@@ -47,8 +74,8 @@
             <xacro:box_inertia m="${m_servo}" x="${d_servo_L}" y="${d_servo_W}" z="${d_servo_H}"/>
         </link>
-        <joint name="parent_to_MJ1_stator" type="fixed">
-            <parent link="${parent}"/>
+        <joint name="servo_mount_to_MJ1_stator" type="fixed">
+            <parent link="servo_mount_link"/>
             <child link="MJ1_stator_link"/>
-            <origin xyz="0 ${d_servo_W/2 - 0.0178} 0" rpy="0 0 0"/>
+            <origin xyz="${d_servo_mount_L/2 - 0.029} ${-d_servo_mount_W/2 + d_servo_W/2 - 0.0178} ${d_servo_mount_H/2 - 0.016}" rpy="0 0 0"/>
         </joint>
         <link name="MJ1_rotor_link"/>
@@ -154,4 +181,5 @@
         </joint>
         <!-- ********************[ GAZEBO CONFIG ]******************** -->
+        <gazebo reference="servo_mount_link"><material>Gazebo/Black</material></gazebo>
         <gazebo reference="MJ1_stator_link"><material>Gazebo/Purple</material></gazebo>
         <gazebo reference="MJ2_stator_link"><material>Gazebo/Purple</material></gazebo>
@@ -159,3 +187,85 @@
         <gazebo reference="sensor_bracket_link"><material>Gazebo/Black</material></gazebo>
     </xacro:macro>
+    <!-- Definition #2: Static Manipulator Mount -->
+    <xacro:macro name="spawn_manip_static" params="parent">
+        <!-- ********************[ PROPERTIES ]******************** -->
+        <!-- Static Mount -->
+        <xacro:property name="d_static_L" value="0.060"/>
+        <xacro:property name="d_static_W" value="0.070"/>
+        <xacro:property name="d_static_H" value="0.070"/>
+        <xacro:property name="m_static" value="?"/>
+        <!-- Sensor Mounting Bracket -->
+        <xacro:property name="d_sensor_bracket_L" value="0.065"/>
+        <xacro:property name="d_sensor_bracket_W" value="0.025"/>
+        <xacro:property name="d_sensor_bracket_H" value="0.055"/>
+        <xacro:property name="m_sensor_bracket" value="0.0081"/>
+        <!-- ********************[ LINKS ]******************** -->
+        <!-- NOTE
+            X = forward/red, Y = left/green, Z = upwards/blue
+        -->
+        <!-- Static Mount -->
+        <link name="static_mount_link">
+            <visual>
+                <origin xyz="${-d_static_L/2 + 0.0049} 0 0" rpy="${PI/2} 0 ${PI/2}"/>
+                <geometry>
+                    <mesh filename="package://libra/meshes/mount-static.stl" scale="0.001 0.001 0.001"/>
+                </geometry>
+                <material name="black"/>
+            </visual>
+            <collision>
+                <origin xyz="0 0 0" rpy="0 0 0"/>
+                <geometry>
+                    <box size="${d_static_L} ${d_static_W} ${d_static_H}"/>
+                </geometry>
+            </collision>
+            <xacro:box_inertia m="${m_static}" x="${d_static_L}" y="${d_static_W}" z="${d_static_H}"/>
+        </link>
+        <joint name="parent_to_static_mount" type="fixed">
+            <parent link="${parent}"/>
+            <child link="static_mount_link"/>
+            <origin xyz="${d_static_L/2} 0 0" rpy="0 0 0"/>
+        </joint>
+        <link name="pseudo_rotor_link"/>
+        <joint name="Static-Manip" type="revolute">
+            <parent link="static_mount_link"/>
+            <child link="pseudo_rotor_link"/>
+            <origin xyz="${d_static_L/2 - 0.023} ${-d_static_W/2 + 0.01} 0" rpy="0 0 0"/>
+            <axis xyz="0 1 0"/>
+            <limit lower="-${PI/2}" upper="${PI/2}" effort="50" velocity="1.5"/>
+        </joint>
+        ---
+        <!-- Sensor Mounting Bracket -->
+        <link name="sensor_bracket_link">
+            <visual>
+                <origin xyz="${d_sensor_bracket_L/2} 0 0" rpy="${PI/2} 0 -${PI/2}"/>
+                <geometry>
+                    <mesh filename="package://libra/meshes/sensor_bracket.stl" scale="0.001 0.001 0.001"/>
+                </geometry>
+                <material name="black"/>
+            </visual>
+            <collision>
+                <origin xyz="0 0 0" rpy="0 0 0"/>
+                <geometry>
+                    <box size="${d_sensor_bracket_L} ${d_sensor_bracket_H} ${d_sensor_bracket_W}"/>
+                </geometry>
+            </collision>
+            <xacro:box_inertia m="${m_sensor_bracket}" x="${d_sensor_bracket_L}" y="${d_sensor_bracket_H}" z="${d_sensor_bracket_W}"/>
+        </link>
+        <joint name="pseudo_rotor_to_sensor_bracket" type="fixed">
+            <parent link="pseudo_rotor_link"/>
+            <child link="sensor_bracket_link"/>
+            <origin xyz="${d_sensor_bracket_L/2 - 0.0125} ${d_sensor_bracket_W} 0" rpy="0 0 0"/>
+        </joint>
+        ---
+        <!-- Outbound Link -->
+        <link name="manip_out_link"/>
+        <joint name="sensor_bracket_to_manip_out" type="fixed">
+            <parent link="sensor_bracket_link"/>
+            <child link="manip_out_link"/>
+            <origin xyz="${d_sensor_bracket_L/2} 0 0" rpy="0 0 0"/>
+        </joint>
+        <!-- ********************[ GAZEBO CONFIG ]******************** -->
+        <gazebo reference="static_mount_link"><material>Gazebo/Black</material></gazebo>
+        <gazebo reference="sensor_bracket_link"><material>Gazebo/Black</material></gazebo>
+    </xacro:macro>
 </robot>

File: ros2_ws/src/libra/models/display_manip.urdf.xacro (robot description, xacro)
@@ -10,3 +10,4 @@
     <link name="base_link"/>
     <xacro:spawn_manip parent="base_link"/>
+    <!-- <xacro:spawn_manip_static parent="base_link"/> -->
 </robot>

File: ros2_ws/src/libra/models/robots/libra1.urdf.xacro (robot description, xacro)
@@ -21,5 +21,6 @@
     <xacro:spawn_2djnt parent="base_link"/>
     <xacro:spawn_arm parent="2djnt_out_arm_link"/>
-    <xacro:spawn_manip parent="arm_out_link"/>
+    <!-- <xacro:spawn_manip parent="arm_out_link"/> -->
+    <xacro:spawn_manip_static parent="arm_out_link"/>
     <xacro:spawn_sensors parent="manip_out_link"/>
 </robot>

Commit message: formatting

File: ros2_ws/src/libra/models/assemblies/arm.urdf.xacro (robot description, xacro)
@@ -144,5 +144,4 @@
         <xacro:joint_subassembly_macro name="J1" parent_name="L1"
             origin_xyz="${d_arm_link_L/2 + d_conn_outer_L/2} 0 0" origin_rpy="0 0 0"/>
-        ---
         <!-- Arm Segment #2 -->
         <xacro:link_macro name="L2_link"/>
@@ -154,5 +153,4 @@
         <xacro:joint_subassembly_macro name="J2" parent_name="L2"
             origin_xyz="${d_arm_link_L/2 + d_conn_outer_L/2} 0 0" origin_rpy="${PI} 0 0"/>
-        ---
         <!-- Arm Segment #3 -->
         <xacro:link_macro name="L3_link"/>
@@ -185,5 +183,4 @@
         <xacro:joint_subassembly_macro name="J3" parent_name="J3_conn_adapter"
             origin_xyz="${d_adapter_L/2 + d_conn_outer_L/2} 0 0" origin_rpy="${PI/2} 0 0"/>
-        ---
         <!-- Arm Segment #4 -->
         <xacro:link_macro name="L4_link"/>

File: ros2_ws/src/libra/models/assemblies/manip.urdf.xacro (robot description, xacro)
@@ -57,5 +57,5 @@
             <origin xyz="${d_servo_mount_L/2} 0 ${0.042 - d_servo_mount_H/2}" rpy="0 0 0"/>
         </joint>
-        <!-- Manipulator Joint #1 (servo) -->
+        <!-- Servo Joint #1 -->
         <link name="MJ1_stator_link">
             <visual>
@@ -87,6 +87,5 @@
             <limit lower="-${PI/2}" upper="${PI/2}" effort="50" velocity="1.5"/>
         </joint>
-        ---
-        <!-- Manipulator Joint #2 (servo w/ bracket) -->
+        <!-- Servo Joint #2 (w/ bracket) -->
         <link name="MJ2_stator_link">
             <visual>
@@ -118,6 +117,5 @@
             <limit lower="-${PI/2}" upper="${PI/2}" effort="50" velocity="1.5"/>
         </joint>
-        ---
-        <!-- Manipulator Joint #3 (servo w/ bracket) -->
+        <!-- Servo Joint #3 (w/ bracket) -->
         <link name="MJ3_stator_link">
             <visual>
@@ -149,5 +147,4 @@
             <limit lower="-${PI/2}" upper="${PI/2}" effort="50" velocity="1.5"/>
         </joint>
-        ---
         <!-- Sensor Mounting Bracket -->
         <link name="sensor_bracket_link">
@@ -172,5 +169,4 @@
             <origin xyz="${d_sensor_bracket_L/2 - 0.0125} ${d_sensor_bracket_W} 0" rpy="0 0 0"/>
         </joint>
-        ---
         <!-- Outbound Link -->
         <link name="manip_out_link"/>
@@ -194,5 +190,5 @@
         <xacro:property name="d_static_W" value="0.070"/>
         <xacro:property name="d_static_H" value="0.070"/>
-        <xacro:property name="m_static" value="?"/>
+        <xacro:property name="m_static" value="0.150"/>
         <!-- Sensor Mounting Bracket -->
         <xacro:property name="d_sensor_bracket_L" value="0.065"/>
@@ -234,5 +230,4 @@
             <limit lower="-${PI/2}" upper="${PI/2}" effort="50" velocity="1.5"/>
         </joint>
-        ---
         <!-- Sensor Mounting Bracket -->
         <link name="sensor_bracket_link">
@@ -257,5 +252,4 @@
             <origin xyz="${d_sensor_bracket_L/2 - 0.0125} ${d_sensor_bracket_W} 0" rpy="0 0 0"/>
         </joint>
-        ---
         <!-- Outbound Link -->
         <link name="manip_out_link"/>

File: ros2_ws/src/libra/models/assemblies/sensor_suite.urdf.xacro (robot description, xacro)
@@ -86,5 +86,4 @@
             <origin xyz="0.006 0 0" rpy="0 ${PI/2} 0"/>  <!-- facing downwards -->
         </joint>
-        ---
         <!-- Camera Mount -->
         <link name="mount_camera_link">

File: ros2_ws/src/libra/models/common/common.urdf.xacro (robot description, xacro)
@@ -7,63 +7,67 @@
 ****************************************************************************-->
 <robot xmlns:xacro="http://www.ros.org/wiki/xacro">
-    <!-- ********************[ PROPERTIES ]******************** -->
-    <xacro:property name="PI" value="3.14159265359"/>
-    <!-- ********************[ MATERIALS ]******************** -->
-    <!-- Colors: Monochrome -->
-    <material name="black">
-        <color rgba="${20/255} ${20/255} ${20/255} 1"/>
-    </material>
-    <material name="gray">
-        <color rgba="${90/255} ${90/255} ${90/255} 1"/>
-    </material>
-    <material name="silver">
-        <color rgba="${170/255} ${170/255} ${170/255} 1"/>
-    </material>
-    <material name="white">
-        <color rgba="${250/255} ${250/255} ${250/255} 1"/>
-    </material>
-    <!-- Colors: Primary & Secondary -->
-    <material name="red">
-        <color rgba="${200/255} ${30/255} ${30/255} 1"/>
-    </material>
-    <material name="yellow">
-        <color rgba="${225/255} ${200/255} ${40/255} 1"/>
-    </material>
-    <material name="blue">
-        <color rgba="${40/255} ${110/255} ${200/255} 1"/>
-    </material>
-    <material name="orange">
-        <color rgba="${220/255} ${110/255} ${40/255} 1"/>
-    </material>
-    <material name="green">
-        <color rgba="${50/255} ${170/255} ${90/255} 1"/>
-    </material>
-    <material name="purple">
-        <color rgba="${150/255} ${50/255} ${200/255} 1"/>
-    </material>
-    <!-- ********************[ MACROS ]******************** -->
-    <xacro:macro name="box_inertia" params="m x y z">
-        <inertial>
-            <mass value="${m}"/>
-            <inertia ixx="${(m/12) * (y*y + z*z)}" ixy="0.0" ixz="0.0"
-                     iyy="${(m/12) * (x*x + z*z)}" iyz="0.0"
-                     izz="${(m/12) * (x*x + y*y)}"/>
-        </inertial>
-    </xacro:macro>
-    <xacro:macro name="cylinder_inertia" params="m r h">
-        <inertial>
-            <mass value="${m}"/>
-            <inertia ixx="${(m/12) * (3*r*r + h*h)}" ixy = "0" ixz = "0"
-                     iyy="${(m/12) * (3*r*r + h*h)}" iyz = "0"
-                     izz="${(m/2) * (r*r)}"/>
-        </inertial>
-    </xacro:macro>
-    <xacro:macro name="sphere_inertia" params="m r">
-        <inertial>
-            <mass value="${m}"/>
-            <inertia ixx="${(2/5) * m * (r*r)}" ixy="0.0" ixz="0.0"
-                    iyy="${(2/5) * m * (r*r)}" iyz="0.0"
-                    izz="${(2/5) * m * (r*r)}"/>
-        </inertial>
-    </xacro:macro>
+    <!-- Prevent duplicate inclusion -->
+    <xacro:unless value="$(optenv COMMON_URDF_INCLUDED false)">
+        <xacro:property name="COMMON_URDF_INCLUDED" value="true"/>
+        <!-- ********************[ PROPERTIES ]******************** -->
+        <xacro:property name="PI" value="3.14159265359"/>
+        <!-- ********************[ MATERIALS ]******************** -->
+        <!-- Colors: Monochrome -->
+        <material name="black">
+            <color rgba="${20/255} ${20/255} ${20/255} 1"/>
+        </material>
+        <material name="gray">
+            <color rgba="${90/255} ${90/255} ${90/255} 1"/>
+        </material>
+        <material name="silver">
+            <color rgba="${170/255} ${170/255} ${170/255} 1"/>
+        </material>
+        <material name="white">
+            <color rgba="${250/255} ${250/255} ${250/255} 1"/>
+        </material>
+        <!-- Colors: Primary & Secondary -->
+        <material name="red">
+            <color rgba="${200/255} ${30/255} ${30/255} 1"/>
+        </material>
+        <material name="yellow">
+            <color rgba="${225/255} ${200/255} ${40/255} 1"/>
+        </material>
+        <material name="blue">
+            <color rgba="${40/255} ${110/255} ${200/255} 1"/>
+        </material>
+        <material name="orange">
+            <color rgba="${220/255} ${110/255} ${40/255} 1"/>
+        </material>
+        <material name="green">
+            <color rgba="${50/255} ${170/255} ${90/255} 1"/>
+        </material>
+        <material name="purple">
+            <color rgba="${150/255} ${50/255} ${200/255} 1"/>
+        </material>
+        <!-- ********************[ MACROS ]******************** -->
+        <xacro:macro name="box_inertia" params="m x y z">
+            <inertial>
+                <mass value="${m}"/>
+                <inertia ixx="${(m/12) * (y*y + z*z)}" ixy="0.0" ixz="0.0"
+                        iyy="${(m/12) * (x*x + z*z)}" iyz="0.0"
+                        izz="${(m/12) * (x*x + y*y)}"/>
+            </inertial>
+        </xacro:macro>
+        <xacro:macro name="cylinder_inertia" params="m r h">
+            <inertial>
+                <mass value="${m}"/>
+                <inertia ixx="${(m/12) * (3*r*r + h*h)}" ixy = "0" ixz = "0"
+                        iyy="${(m/12) * (3*r*r + h*h)}" iyz = "0"
+                        izz="${(m/2) * (r*r)}"/>
+            </inertial>
+        </xacro:macro>
+        <xacro:macro name="sphere_inertia" params="m r">
+            <inertial>
+                <mass value="${m}"/>
+                <inertia ixx="${(2/5) * m * (r*r)}" ixy="0.0" ixz="0.0"
+                        iyy="${(2/5) * m * (r*r)}" iyz="0.0"
+                        izz="${(2/5) * m * (r*r)}"/>
+            </inertial>
+        </xacro:macro>
+    </xacro:unless>
 </robot>

File: ros2_ws/src/libra/models/display_manip.urdf.xacro (robot description, xacro)
@@ -9,5 +9,5 @@
     <xacro:include filename="$(find libra)/models/assemblies/manip.urdf.xacro"/>
     <link name="base_link"/>
-    <xacro:spawn_manip parent="base_link"/>
-    <!-- <xacro:spawn_manip_static parent="base_link"/> -->
+    <!-- <xacro:spawn_manip parent="base_link"/> -->
+    <xacro:spawn_manip_static parent="base_link"/>
 </robot>

File: ros2_ws/src/libra/models/robots/libra1_no_manip.urdf.xacro (robot description, xacro)
@@ -2,5 +2,5 @@
 <!--***************************************************************************
 /// @file   libra1_no_manip.urdf.xacro
-/// @brief  LIBRA-I (w/o customization) model constructor.
+/// @brief  LIBRA-I (base 5-DoF arm only) model constructor.
 ///
 /// @author brice.c.aa
